File: hardware/r0ket/r0ket_v2.sch (EAGLE design)
At the start: 89 parts, among them IC1 MCP1700, IC2 LPC1343, IC3 AT45DB041D, IC4 NRF24L01SMD, IC5 MCP73833, IC6 TB62737, M0DULA M06X2PTH, M0DULB M06X2PTH, Q1 Q12M-SMD-S, Q2 3.2X2.5CRYSTAL, SW1 JS102011SAQN, T1 SI2301DS, T3 SI2301DS, T4 SI2301DS, T5 SI2301DS, T6 SI2301DS, X1 MICROUSB, X1_ JST-PH3, X2 NOKIA

Commit message: removed a lot of components
Parts:
- removed BTN1: MCMT5-F-V, badge:MCMT5-F-V
- removed C24, C6: 100nF, rcl:C-EUC0402K
- removed C5: 10uF, rcl:C-EUC0805K
- removed D2: SS14, diode:DIODE-SMB
- removed IC2: LPC1343, microbuilder:LPC1343_QFP
- removed IC3: AT45DB041D, SparkFun:AT45DB041B
- removed IC6: TB62737, badge:TB62737
- removed JP1, JP2: (no value), SparkFun:M07
- removed L1: 4u7, badge:L-EU
- removed M0DULA, M0DULB: M06X2PTH, con-lstb:MA06-2
- removed R1: 1k5, rcl:R-EU_R0603
- removed R10: 15, rcl:R-EU_R0603
- removed R18, R19: 4k7, rcl:R-EU_R0603
- removed R20: 100k, rcl:R-EU_R0603
- removed R21: 10k, rcl:R-EU_R0603
- removed T3, T4: SI2301DS, transistor-small-signal:BSS84
- removed X2: NOKIA, badge:NOKIA
Connections:
- removed net BTN0: BTN1.LEFT, IC2.PIO0_1/CLKOUT/CT32B0_MAT2/USB_FTOGGLE
- removed net BTN1: BTN1.RIGHT, IC2.PIO2_9
- removed net BTN2: BTN1.DOWN, IC2.PIO2_6
- removed net BTN3: BTN1.UP, IC2.PIO3_3
- removed net BTN4: BTN1.DUMMY, IC2.PIO2_7
- removed net BUSINT: IC2.PIO3_0, M0DULA.11, M0DULB.11
- removed net CS_DF: IC2.PIO2_0/DTR, IC3.CS
- removed net HB0: IC2.SWDIO/PIO1_3/AD4/CT32B1_MAT2, JP2.4
- removed net HB1: IC2.SWCLK/PIO0_10/SCK/CT16B0_MAT2, JP2.5
- removed net HB2: IC2.TDO/PIO1_1/AD2/CT32B1_MAT0, JP2.6
- removed net HB3: IC2.PIO0_2/SSEL/CT16B0_CAP0, JP1.4
- removed net HB4: IC2.PIO1_4/AD5/CT32B1_MAT3/WAKEUP, JP1.5, R20.1
- removed net HB5: IC2.TRST/PIO1_2/AD3/CT32B1_MAT1, JP1.6
- removed net LCD_BL: IC2.PIO1_9/CT16B1_MAT0, IC6.!SHDN
- removed net LCD_BLEN: IC2.RESET/PIO0_0, R21.1, T3.G
- removed net LCD_CS: IC2.PIO2_1/DSR, X2.CS
- removed net LCD_RST: IC2.PIO2_2/DCD, X2.RESET
- removed net LED+: C6.2, D2.C, IC6.OVD, X2.LED+
- removed net LED-: IC6.FB, R10.2, X2.LED-
- removed net N$14: D2.A, IC6.SW, L1.2
- removed net N$20: R1.1, T4.D
- removed net SCL: IC2.PIO0_4/SCL, M0DULA.9, M0DULB.9, R19.1
- removed net SDA: IC2.PIO0_5/SDA, M0DULA.7, M0DULB.7, R18.2
- removed net SS0: IC2.PIO2_5, M0DULA.6
- removed net SS1: IC2.PIO2_4, M0DULA.8
- removed net SS2: IC2.PIO2_8, M0DULA.10
- removed net SS4: IC2.PIO3_1, M0DULB.8
- removed net SS5: IC2.PIO2_10, M0DULB.10
- removed net USB_CONNECT: IC2.PIO0_6/USB_CONNECT/SCK, T4.G
- removed net VCC_LCD: C5.2, IC6.VCC, L1.1, T3.D
- net +3V3: no longer IC2.VDD(3V3), IC2.VDD(IO), R18.1, R19.2, R20.2, T4.S
- net +3V3_EXP: no longer C24.2, IC3.RST, IC3.VCC, IC3.WP, JP1.1, JP2.1, M0DULA.1, M0DULB.1, X2.VDD, X2.VIO
- net CE: no longer IC2.PIO1_5/RTS/CT32B0_CAP0
- net CHRG_STAT: no longer IC2.PIO2_3/RI
- net CSN: no longer IC2.PIO1_10/AD6/CT16B1_MAT1
- net D+: no longer R1.2
- net GND: no longer BTN1.COMMON, BTN1.TAB1, BTN1.TAB2, C24.1, C5.1, C6.1, IC2.VSS, IC2.VSSIO, IC3.GND, IC6.GND, JP1.2, JP2.2, M0DULA.5, M0DULB.5, R10.1, X2.GND, X2.NC
- net IRQ: no longer IC2.PIO0_7/CTS
- net LED0: no longer IC2.TDI/PIO0_11/AD0/CT32B0_MAT3
- net LED1: no longer IC2.PIO1_7/TXD/CT32B0_MAT1, JP1.7
- net LED2: no longer IC2.PIO1_6/RXD/CT32B0_MAT0, JP2.7
- net LED3: no longer IC2.PIO1_11/AD7
- net MISO: no longer IC2.PIO0_8/MISO/CT16B0_MAT0, IC3.SO, M0DULA.2, M0DULB.2
- net MOSI: no longer IC2.PIO0_9/MOSI/CT16B0_MAT1/SWO, IC3.SI, M0DULA.3, M0DULB.3, X2.SDA
- net N$1: no longer IC2.XTALIN
- net N$3: no longer IC2.XTALOUT
- net POWER_GOOD: no longer IC2.PIO1_8/CT16B1_CAP0
- net SCK: no longer IC2.PIO2_11/SCK, IC3.SCK, M0DULA.4, M0DULB.4, X2.CLK
- net SS3: no longer IC2.PIO3_2, M0DULB.6
- net USB_DM: no longer IC2.USB_DM
- net USB_DP: no longer IC2.USB_DP
- net USB_VBUS: no longer IC2.PIO0_3/USB_VBUS
- net VCC_EXP: no longer JP1.3, JP2.3, M0DULA.12, M0DULB.12, R21.2, T3.S
- net VOLTAGE: no longer IC2.TMS/PIO1_0/AD1/CT32B1_CAP0
Other:
- note removed: "4MBit DATAFLASH"
- note removed: "HACKER BUS"
- note removed: "M0DUL BUS"
