File: eagle/lun1k.sch (EAGLE design)
At the start: 100 parts, among them IC1 LTC3558, IC3 STM32F405RGT, IC4 NRF24L01SMD, J2 XF2-3015-1LW, Q1 Q12M-SMD-S, Q2 3.2X2.5CRYSTAL, SW1 JS102011SAQN, SW2 SWITCH_MCTAEF, SW3 SWITCH_MCTAEF, SW4 SWITCH_MCTAEF, T5 SI2301DS, T6 SI2301DS, U1 N35P112, X1 MICROUSB, X1_ JST-PH3

Commit message: routing
Connections:
- new net D2: J2-19.MS
- new net D3: J2-20.MS
- new net D4: J2-21.MS
- new net D5: J2-22.MS
- new net D6: IC3.PB14, J2-23.MS
- new net D7: IC3.PB13, J2-24.MS
- new net D8: IC3.PB12, J2-25.MS
- new net E: J2-16.MS
- new net R/W: J2-15.MS
- net +3V3: now also J2-13.MS, J2-14.MS
- net EN2: no longer IC3.PB12
- net GND: no longer J2-13.MS, J2-14.MS, J2-15.MS, J2-16.MS
- net N$23: no longer IC3.PB13
Changed lines of the file:
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@@
 </part>
 <part name="GND21" library="supply1" deviceset="GND" device=""/>
-<part name="GND30" library="supply1" deviceset="GND" device=""/>
-<part name="GND31" library="supply1" deviceset="GND" device=""/>
-<part name="GND32" library="supply1" deviceset="GND" device=""/>
-<part name="GND33" library="supply1" deviceset="GND" device=""/>
 <part name="C36" library="SparkFun-Capacitors" deviceset="CAP" device="0402-CAP" value="100nF"/>
 <part name="C37" library="SparkFun-Capacitors" deviceset="CAP" device="0402-CAP" value="100nF"/>
@@
 <instance part="J2" gate="-30" x="99.06" y="185.42" rot="MR180"/>
 <instance part="GND21" gate="1" x="63.5" y="139.7" rot="R270"/>
-<instance part="GND30" gate="1" x="63.5" y="142.24" rot="R270"/>
-<instance part="GND31" gate="1" x="63.5" y="144.78" rot="R270"/>
-<instance part="GND32" gate="1" x="63.5" y="147.32" rot="R270"/>
-<instance part="GND33" gate="1" x="63.5" y="149.86" rot="R270"/>
 <instance part="C36" gate="G$1" x="134.62" y="76.2" rot="R270"/>
 <instance part="C37" gate="G$1" x="78.74" y="96.52" rot="R180"/>
@@
 </segment>
 <segment>
-<wire x1="76.2" y1="142.24" x2="66.04" y2="142.24" width="0.1524" layer="91"/>
-<wire x1="76.2" y1="142.24" x2="96.52" y2="142.24" width="0.1524" layer="91"/>
-<label x="66.04" y="142.24" size="1.778" layer="95"/>
-<pinref part="J2" gate="-13" pin="MS"/>
-<pinref part="GND30" gate="1" pin="GND"/>
-</segment>
-<segment>
-<wire x1="76.2" y1="144.78" x2="66.04" y2="144.78" width="0.1524" layer="91"/>
-<wire x1="96.52" y1="144.78" x2="76.2" y2="144.78" width="0.1524" layer="91"/>
-<label x="66.04" y="144.78" size="1.778" layer="95"/>
-<pinref part="J2" gate="-14" pin="MS"/>
-<pinref part="GND31" gate="1" pin="GND"/>
-</segment>
-<segment>
-<wire x1="76.2" y1="147.32" x2="66.04" y2="147.32" width="0.1524" layer="91"/>
-<wire x1="76.2" y1="147.32" x2="96.52" y2="147.32" width="0.1524" layer="91"/>
-<label x="66.04" y="147.32" size="1.778" layer="95"/>
-<pinref part="J2" gate="-15" pin="MS"/>
-<pinref part="GND32" gate="1" pin="GND"/>
-</segment>
-<segment>
-<wire x1="76.2" y1="149.86" x2="66.04" y2="149.86" width="0.1524" layer="91"/>
-<wire x1="96.52" y1="149.86" x2="76.2" y2="149.86" width="0.1524" layer="91"/>
-<label x="66.04" y="149.86" size="1.778" layer="95"/>
-<pinref part="J2" gate="-16" pin="MS"/>
-<pinref part="GND33" gate="1" pin="GND"/>
-</segment>
-<segment>
 <wire x1="76.2" y1="139.7" x2="66.04" y2="139.7" width="0.1524" layer="91"/>
 <wire x1="96.52" y1="139.7" x2="76.2" y2="139.7" width="0.1524" layer="91"/>
@@
 <pinref part="U1" gate="G$1" pin="VDDP"/>
 <pinref part="U1" gate="G$1" pin="VDD"/>
+</segment>
+<segment>
+<wire x1="66.04" y1="142.24" x2="96.52" y2="142.24" width="0.1524" layer="91"/>
+<label x="66.04" y="142.24" size="1.778" layer="95"/>
+<pinref part="J2" gate="-13" pin="MS"/>
+</segment>
+<segment>
+<wire x1="96.52" y1="144.78" x2="66.04" y2="144.78" width="0.1524" layer="91"/>
+<label x="66.04" y="144.78" size="1.778" layer="95"/>
+<pinref part="J2" gate="-14" pin="MS"/>
 </segment>
 </net>
@@
 <wire x1="416.56" y1="55.88" x2="416.56" y2="17.78" width="0.1524" layer="91"/>
 <wire x1="416.56" y1="17.78" x2="137.16" y2="17.78" width="0.1524" layer="91"/>
-<wire x1="137.16" y1="17.78" x2="137.16" y2="40.64" width="0.1524" layer="91"/>
-<pinref part="IC3" gate="G$1" pin="PB13"/>
-<wire x1="137.16" y1="40.64" x2="132.08" y2="40.64" width="0.1524" layer="91"/>
 </segment>
 </net>
@@
 <pinref part="IC1" gate="G$1" pin="EN2"/>
 <pinref part="R24" gate="G$1" pin="2"/>
-<pinref part="IC3" gate="G$1" pin="PB12"/>
 <wire x1="482.6" y1="27.94" x2="132.08" y2="27.94" width="0.1524" layer="91"/>
-<wire x1="132.08" y1="27.94" x2="132.08" y2="38.1" width="0.1524" layer="91"/>
 </segment>
 </net>
@@
 </segment>
 </net>
+<net name="D2" class="0">
+<segment>
+<pinref part="J2" gate="-19" pin="MS"/>
+<wire x1="96.52" y1="157.48" x2="66.04" y2="157.48" width="0.1524" layer="91"/>
+<label x="66.04" y="157.48" size="1.778" layer="95"/>
+</segment>
+</net>
+<net name="D3" class="0">
+<segment>
+<pinref part="J2" gate="-20" pin="MS"/>
+<wire x1="96.52" y1="160.02" x2="66.04" y2="160.02" width="0.1524" layer="91"/>
+<label x="66.04" y="160.02" size="1.778" layer="95"/>
+</segment>
+</net>
+<net name="D4" class="0">
+<segment>
+<pinref part="J2" gate="-21" pin="MS"/>
+<wire x1="96.52" y1="162.56" x2="66.04" y2="162.56" width="0.1524" layer="91"/>
+<label x="66.04" y="162.56" size="1.778" layer="95"/>
+</segment>
+</net>
+<net name="D5" class="0">
+<segment>
+<pinref part="J2" gate="-22" pin="MS"/>
+<wire x1="96.52" y1="165.1" x2="66.04" y2="165.1" width="0.1524" layer="91"/>
+<label x="66.04" y="165.1" size="1.778" layer="95"/>
+</segment>
+</net>
+<net name="D6" class="0">
+<segment>
+<pinref part="J2" gate="-23" pin="MS"/>
+<wire x1="96.52" y1="167.64" x2="66.04" y2="167.64" width="0.1524" layer="91"/>
+<label x="66.04" y="167.64" size="1.778" layer="95"/>
+</segment>
+<segment>
+<pinref part="IC3" gate="G$1" pin="PB14"/>
+<wire x1="132.08" y1="43.18" x2="142.24" y2="43.18" width="0.1524" layer="91"/>
+<label x="137.16" y="43.18" size="1.778" layer="95"/>
+</segment>
+</net>
+<net name="D7" class="0">
+<segment>
+<pinref part="J2" gate="-24" pin="MS"/>
+<wire x1="96.52" y1="170.18" x2="66.04" y2="170.18" width="0.1524" layer="91"/>
+<label x="66.04" y="170.18" size="1.778" layer="95"/>
+</segment>
+<segment>
+<pinref part="IC3" gate="G$1" pin="PB13"/>
+<wire x1="132.08" y1="40.64" x2="142.24" y2="40.64" width="0.1524" layer="91"/>
+<label x="137.16" y="40.64" size="1.778" layer="95"/>
+</segment>
+</net>
+<net name="D8" class="0">
+<segment>
+<pinref part="J2" gate="-25" pin="MS"/>
+<wire x1="96.52" y1="172.72" x2="66.04" y2="172.72" width="0.1524" layer="91"/>
+<label x="66.04" y="172.72" size="1.778" layer="95"/>
+</segment>
+<segment>
+<pinref part="IC3" gate="G$1" pin="PB12"/>
+<wire x1="132.08" y1="38.1" x2="142.24" y2="38.1" width="0.1524" layer="91"/>
+<label x="137.16" y="38.1" size="1.778" layer="95"/>
+</segment>
+</net>
+<net name="R/W" class="2">
+<segment>
+<wire x1="66.04" y1="147.32" x2="96.52" y2="147.32" width="0.1524" layer="91"/>
+<label x="66.04" y="147.32" size="1.778" layer="95"/>
+<pinref part="J2" gate="-15" pin="MS"/>
+</segment>
+</net>
+<net name="E" class="2">
+<segment>
+<wire x1="96.52" y1="149.86" x2="66.04" y2="149.86" width="0.1524" layer="91"/>
+<label x="66.04" y="149.86" size="1.778" layer="95"/>
+<pinref part="J2" gate="-16" pin="MS"/>
+</segment>
+</net>

Commit message: routing
Connections:
- net D/C: now also IC3.PC5
- net D0: now also IC3.PB10
- net D1: now also IC3.PB11
- net D2: now also IC3.PC9
- net D3: now also IC3.PC8
- net D4: now also IC3.PC7
- net D5: now also IC3.PB15
- net E: now also IC3.PB1
- net GND: no longer IC3.PB11
- net R/W: now also IC3.PB0
- net RES: now also IC3.PC4
Changed lines of the file:
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@@
 <part name="C41" library="SparkFun" deviceset="CAP" device="0805" value="2,2µF"/>
 <part name="GND42" library="supply1" deviceset="GND" device=""/>
-<part name="GND43" library="supply1" deviceset="GND" device=""/>
 <part name="GND44" library="supply1" deviceset="GND" device=""/>
 <part name="GND45" library="supply1" deviceset="GND" device=""/>
@@
 <instance part="C41" gate="G$1" x="137.16" y="73.66" rot="R270"/>
 <instance part="GND42" gate="1" x="142.24" y="73.66" rot="R90"/>
-<instance part="GND43" gate="1" x="111.76" y="20.32"/>
 <instance part="GND44" gate="1" x="109.22" y="93.98" rot="R180"/>
 <instance part="GND45" gate="1" x="96.52" y="93.98" rot="R180"/>
@@
 </segment>
 <segment>
-<pinref part="IC3" gate="G$1" pin="PB11"/>
-<pinref part="GND43" gate="1" pin="GND"/>
-</segment>
-<segment>
 <pinref part="IC3" gate="G$1" pin="PB2"/>
 <pinref part="GND46" gate="1" pin="GND"/>
@@
 <pinref part="J2" gate="-10" pin="MS"/>
 </segment>
+<segment>
+<pinref part="IC3" gate="G$1" pin="PC4"/>
+<wire x1="96.52" y1="22.86" x2="96.52" y2="7.62" width="0.1524" layer="91"/>
+<label x="96.52" y="7.62" size="1.778" layer="95" rot="R90"/>
+</segment>
 </net>
 <net name="D/C" class="0">
@@
 <pinref part="J2" gate="-11" pin="MS"/>
 </segment>
+<segment>
+<pinref part="IC3" gate="G$1" pin="PC5"/>
+<wire x1="99.06" y1="22.86" x2="99.06" y2="7.62" width="0.1524" layer="91"/>
+<label x="99.06" y="7.62" size="1.778" layer="95" rot="R90"/>
+</segment>
 </net>
 <net name="D1" class="0">
@@
 <label x="66.04" y="154.94" size="1.778" layer="95"/>
 <pinref part="J2" gate="-18" pin="MS"/>
+</segment>
+<segment>
+<pinref part="IC3" gate="G$1" pin="PB11"/>
+<wire x1="111.76" y1="22.86" x2="111.76" y2="7.62" width="0.1524" layer="91"/>
+<label x="111.76" y="7.62" size="1.778" layer="95" rot="R90"/>
 </segment>
 </net>
@@
 <label x="66.04" y="152.4" size="1.778" layer="95"/>
 <pinref part="J2" gate="-17" pin="MS"/>
+</segment>
+<segment>
+<pinref part="IC3" gate="G$1" pin="PB10"/>
+<wire x1="109.22" y1="22.86" x2="109.22" y2="7.62" width="0.1524" layer="91"/>
+<label x="109.22" y="7.62" size="1.778" layer="95" rot="R90"/>
 </segment>
 </net>
@@
 <label x="66.04" y="157.48" size="1.778" layer="95"/>
 </segment>
+<segment>
+<pinref part="IC3" gate="G$1" pin="PC9"/>
+<wire x1="132.08" y1="55.88" x2="142.24" y2="55.88" width="0.1524" layer="91"/>
+<label x="137.16" y="55.88" size="1.778" layer="95"/>
+</segment>
 </net>
 <net name="D3" class="0">
@@
 <label x="66.04" y="160.02" size="1.778" layer="95"/>
 </segment>
+<segment>
+<pinref part="IC3" gate="G$1" pin="PC8"/>
+<wire x1="132.08" y1="53.34" x2="142.24" y2="53.34" width="0.1524" layer="91"/>
+<label x="137.16" y="53.34" size="1.778" layer="95"/>
+</segment>
 </net>
 <net name="D4" class="0">
@@
 <label x="66.04" y="162.56" size="1.778" layer="95"/>
 </segment>
+<segment>
+<pinref part="IC3" gate="G$1" pin="PC7"/>
+<wire x1="132.08" y1="50.8" x2="142.24" y2="50.8" width="0.1524" layer="91"/>
+<label x="137.16" y="50.8" size="1.778" layer="95"/>
+</segment>
 </net>
 <net name="D5" class="0">
@@
 <label x="66.04" y="165.1" size="1.778" layer="95"/>
 </segment>
+<segment>
+<pinref part="IC3" gate="G$1" pin="PB15"/>
+<wire x1="132.08" y1="45.72" x2="142.24" y2="45.72" width="0.1524" layer="91"/>
+<label x="137.16" y="45.72" size="1.778" layer="95"/>
+</segment>
 </net>
 <net name="D6" class="0">
@@
 <pinref part="J2" gate="-15" pin="MS"/>
 </segment>
+<segment>
+<pinref part="IC3" gate="G$1" pin="PB0"/>
+<wire x1="101.6" y1="22.86" x2="101.6" y2="7.62" width="0.1524" layer="91"/>
+<label x="101.6" y="7.62" size="1.778" layer="95" rot="R90"/>
+</segment>
 </net>
 <net name="E" class="2">
@@
 <pinref part="J2" gate="-16" pin="MS"/>
 </segment>
-</net>
+<segment>
+<pinref part="IC3" gate="G$1" pin="PB1"/>
+<wire x1="104.14" y1="22.86" x2="104.14" y2="7.62" width="0.1524" layer="91"/>
+<label x="104.14" y="7.62" size="1.778" layer="95" rot="R90"/>
+</segment>
+</net>
