File: eagle/lun1k.sch (EAGLE design)
At the start: 94 parts, among them IC1 LTC3558, IC3 STM32F405RGT, IC4 NRF24L01SMD, J2 XF2-3015-1LW, Q1 Q12M-SMD-S, Q2 3.2X2.5CRYSTAL, SW1 JS102011SAQN, SW2 SWITCH_MCTAEF, SW3 SWITCH_MCTAEF, SW4 SWITCH_MCTAEF, U1 N35P112, X1 MICROUSB, X1_ JST-PH3

Commit message: routing
Connections:
- net LED1: now also IC3.PD2
- net LED3: now also IC3.PB3
Changed lines of the file:
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@@
 <net name="LED1" class="0">
 <segment>
-<wire x1="152.4" y1="73.66" x2="162.56" y2="73.66" width="0.1524" layer="91"/>
-<label x="160.02" y="73.66" size="1.778" layer="95"/>
+<wire x1="104.14" y1="91.44" x2="104.14" y2="101.6" width="0.1524" layer="91"/>
+<label x="104.14" y="93.98" size="1.778" layer="95" rot="R90"/>
+<pinref part="IC3" gate="G$1" pin="PD2"/>
 </segment>
 <segment>
@@
 </segment>
 <segment>
-<wire x1="152.4" y1="63.5" x2="162.56" y2="63.5" width="0.1524" layer="91"/>
-<label x="160.02" y="63.5" size="1.778" layer="95"/>
+<wire x1="101.6" y1="91.44" x2="101.6" y2="101.6" width="0.1524" layer="91"/>
+<label x="101.6" y="93.98" size="1.778" layer="95" rot="R90"/>
+<pinref part="IC3" gate="G$1" pin="PB3"/>
 </segment>
 </net>

Commit message: routing
Connections:
- net SCL: now also IC3.PB6
- net SDA: now also IC3.PB7
- net SW3: now also IC3.PB4; no longer IC3.PB7
Other:
- note removed: "POWER SWITCH"
- moved on the sheet: C1, C11, C12, C2, C3, C4, C7, C8, L5, R12, R18, R19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

Commit message: routing
Connections:
- net EN2: now also IC3.PA1; no longer IC3.PA0
- net SW4: now also IC3.PA0; no longer IC3.PC13
- net VOLTAGE: now also IC3.PA3
Changed lines of the file:
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@@
 <pinref part="R6" gate="G$1" pin="1"/>
+</segment>
+<segment>
+<pinref part="IC3" gate="G$1" pin="PA3"/>
+<wire x1="78.74" y1="22.86" x2="78.74" y2="15.24" width="0.1524" layer="91"/>
+<label x="78.74" y="15.24" size="1.778" layer="95" rot="R90"/>
 </segment>
 </net>
@@
 </segment>
 <segment>
-<pinref part="IC3" gate="G$1" pin="PA0"/>
-<wire x1="63.5" y1="43.18" x2="53.34" y2="43.18" width="0.1524" layer="91"/>
-<label x="53.34" y="43.18" size="1.778" layer="95"/>
+<label x="53.34" y="40.64" size="1.778" layer="95"/>
+<wire x1="58.42" y1="40.64" x2="53.34" y2="40.64" width="0.1524" layer="91"/>
+<pinref part="IC3" gate="G$1" pin="PA1"/>
+<wire x1="58.42" y1="40.64" x2="63.5" y2="40.64" width="0.1524" layer="91"/>
 </segment>
 </net>
@@
 <wire x1="162.56" y1="187.96" x2="167.64" y2="187.96" width="0.1524" layer="91"/>
 <label x="165.1" y="187.96" size="1.778" layer="95"/>
-<wire x1="58.42" y1="73.66" x2="63.5" y2="73.66" width="0.1524" layer="91"/>
-<label x="58.42" y="73.66" size="1.778" layer="95"/>
-<pinref part="IC3" gate="G$1" pin="PC13"/>
-</segment>
-</net>
+</segment>
+<segment>
+<pinref part="IC3" gate="G$1" pin="PA0"/>
+<wire x1="63.5" y1="43.18" x2="53.34" y2="43.18" width="0.1524" layer="91"/>
+<label x="53.34" y="43.18" size="1.778" layer="95"/>
+</segment>
+</net>

Commit message: routing
Parts:
- added C25: 100nF, SparkFun-Capacitors:CAP0402-CAP
- added R4: 680k, SparkFun-Resistors:RESISTOR0402-RES
Connections:
- new net N$15: C25.1, IC3.VDDA, R4.1
- net +3V3: now also R4.2
- net GND: now also C25.2, IC3.VSSA
Changed lines of the file:
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@@
 <part name="GND1" library="SparkFun" deviceset="GND" device=""/>
 <part name="GND10" library="supply1" deviceset="GND" device=""/>
+<part name="GND30" library="supply1" deviceset="GND" device=""/>
+<part name="C25" library="SparkFun-Capacitors" deviceset="CAP" device="0402-CAP" value="100nF"/>
+<part name="R4" library="SparkFun-Resistors" deviceset="RESISTOR" device="0402-RES" value="680k"/>
+<part name="GND31" library="supply1" deviceset="GND" device=""/>
+<part name="+3V2" library="supply1" deviceset="+3V3" device=""/>
 </parts>
 <sheets>
@@
 <instance part="GND1" gate="1" x="447.04" y="208.28"/>
 <instance part="GND10" gate="1" x="63.5" y="172.72" rot="R270"/>
+<instance part="GND30" gate="1" x="48.26" y="48.26" rot="R270"/>
+<instance part="C25" gate="G$1" x="43.18" y="40.64"/>
+<instance part="R4" gate="G$1" x="38.1" y="45.72" rot="R180"/>
+<instance part="GND31" gate="1" x="43.18" y="35.56"/>
+<instance part="+3V2" gate="G$1" x="30.48" y="45.72" rot="R90"/>
 </instances>
 <busses>
@@
 <pinref part="GND10" gate="1" pin="GND"/>
 </segment>
+<segment>
+<pinref part="GND30" gate="1" pin="GND"/>
+<pinref part="IC3" gate="G$1" pin="VSSA"/>
+<wire x1="50.8" y1="48.26" x2="63.5" y2="48.26" width="0.1524" layer="91"/>
+</segment>
+<segment>
+<pinref part="C25" gate="G$1" pin="2"/>
+<pinref part="GND31" gate="1" pin="GND"/>
+</segment>
 </net>
 <net name="+5V" class="1">
@@
 <pinref part="+3V1" gate="G$1" pin="+3V3"/>
 <wire x1="134.62" y1="63.5" x2="132.08" y2="63.5" width="0.1524" layer="91"/>
+</segment>
+<segment>
+<pinref part="R4" gate="G$1" pin="2"/>
+<pinref part="+3V2" gate="G$1" pin="+3V3"/>
 </segment>
 </net>
@@
 </segment>
 </net>
+<net name="N$15" class="0">
+<segment>
+<pinref part="IC3" gate="G$1" pin="VDDA"/>
+<wire x1="63.5" y1="45.72" x2="43.18" y2="45.72" width="0.1524" layer="91"/>
+<pinref part="C25" gate="G$1" pin="1"/>
+<pinref part="R4" gate="G$1" pin="1"/>
+<junction x="43.18" y="45.72"/>
+</segment>
+</net>

Commit message: routing
Parts:
- removed R21: 10k, SparkFun:RESISTOR0402-RES
Connections:
- net 3.3V: no longer R21.2
- net SWITCHN: now also IC3.PC13; no longer R21.1
Changed lines of the file:
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@@
 <part name="P+8" library="SparkFun" deviceset="3.3V" device=""/>
 <part name="GND12" library="SparkFun" deviceset="GND" device=""/>
-<part name="R21" library="SparkFun" deviceset="RESISTOR" device="0402-RES" value="10k"/>
 <part name="R26" library="SparkFun" deviceset="RESISTOR" device="0402-RES" value="10k"/>
 <part name="R27" library="SparkFun" deviceset="RESISTOR" device="0402-RES" value="10k"/>
@@
 <instance part="P+8" gate="G$1" x="444.5" y="233.68"/>
 <instance part="GND12" gate="1" x="485.14" y="208.28"/>
-<instance part="R21" gate="G$1" x="454.66" y="167.64" rot="R90"/>
 <instance part="R26" gate="G$1" x="464.82" y="167.64" rot="R90"/>
 <instance part="R27" gate="G$1" x="474.98" y="167.64" rot="R90"/>
@@
 <junction x="474.98" y="175.26"/>
 <pinref part="P+9" gate="G$1" pin="3.3V"/>
-<pinref part="R21" gate="G$1" pin="2"/>
 <pinref part="R26" gate="G$1" pin="2"/>
 <pinref part="R27" gate="G$1" pin="2"/>
@@
 </segment>
 <segment>
-<wire x1="424.18" y1="154.94" x2="454.66" y2="154.94" width="0.1524" layer="91"/>
-<wire x1="454.66" y1="154.94" x2="454.66" y2="162.56" width="0.1524" layer="91"/>
-<label x="426.72" y="154.94" size="1.778" layer="95" font="vector"/>
-<pinref part="R21" gate="G$1" pin="1"/>
-</segment>
-</net>
+<pinref part="IC3" gate="G$1" pin="PC13"/>
+<wire x1="63.5" y1="73.66" x2="55.88" y2="73.66" width="0.1524" layer="91"/>
+<label x="55.88" y="73.66" size="1.778" layer="95"/>
+</segment>
+</net>

Commit message: routing
Parts:
- removed R26: 10k, SparkFun:RESISTOR0402-RES
Connections:
- removed net 3.3V: R26.2, R27.2, R28.2, R29.2
- net +3V3: now also R27.2, R28.2, R29.2
- net INTN: now also IC3.PC0; no longer R26.1
Other:
- moved on the sheet: R27, R28, R29
Changed lines of the file:
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@@
 <part name="P+8" library="SparkFun" deviceset="3.3V" device=""/>
 <part name="GND12" library="SparkFun" deviceset="GND" device=""/>
-<part name="R26" library="SparkFun" deviceset="RESISTOR" device="0402-RES" value="10k"/>
 <part name="R27" library="SparkFun" deviceset="RESISTOR" device="0402-RES" value="10k"/>
-<part name="P+9" library="SparkFun" deviceset="3.3V" device=""/>
 <part name="R28" library="SparkFun" deviceset="RESISTOR" device="0402-RES" value="10k"/>
 <part name="R29" library="SparkFun" deviceset="RESISTOR" device="0402-RES" value="10k"/>
@@
 <instance part="P+8" gate="G$1" x="444.5" y="233.68"/>
 <instance part="GND12" gate="1" x="485.14" y="208.28"/>
-<instance part="R26" gate="G$1" x="464.82" y="167.64" rot="R90"/>
-<instance part="R27" gate="G$1" x="474.98" y="167.64" rot="R90"/>
-<instance part="P+9" gate="G$1" x="444.5" y="177.8"/>
-<instance part="R28" gate="G$1" x="485.14" y="167.64" rot="R90"/>
-<instance part="R29" gate="G$1" x="495.3" y="167.64" rot="R90"/>
+<instance part="R27" gate="G$1" x="436.88" y="220.98" rot="R180"/>
+<instance part="R28" gate="G$1" x="436.88" y="226.06" rot="R180"/>
+<instance part="R29" gate="G$1" x="436.88" y="223.52" rot="R180"/>
 <instance part="SW2" gate="G$1" x="157.48" y="172.72" smashed="yes" rot="MR0">
 <attribute name="NAME" x="149.225" y="168.91" size="1.778" layer="95" rot="MR0"/>
@@
 <pinref part="U1" gate="G$1" pin="VDDP"/>
 <pinref part="U1" gate="G$1" pin="VDD"/>
+<pinref part="R27" gate="G$1" pin="2"/>
+<pinref part="R29" gate="G$1" pin="2"/>
+<wire x1="431.8" y1="220.98" x2="431.8" y2="223.52" width="0.1524" layer="91"/>
+<pinref part="R28" gate="G$1" pin="2"/>
+<wire x1="431.8" y1="223.52" x2="431.8" y2="226.06" width="0.1524" layer="91"/>
+<junction x="431.8" y="223.52"/>
+<wire x1="431.8" y1="226.06" x2="431.8" y2="231.14" width="0.1524" layer="91"/>
+<junction x="431.8" y="226.06"/>
+<wire x1="444.5" y1="231.14" x2="431.8" y2="231.14" width="0.1524" layer="91"/>
 </segment>
 <segment>
@@
 </segment>
 </net>
-<net name="3.3V" class="0">
-<segment>
-<wire x1="444.5" y1="177.8" x2="444.5" y2="175.26" width="0.1524" layer="91"/>
-<wire x1="444.5" y1="175.26" x2="444.5" y2="172.72" width="0.1524" layer="91"/>
-<wire x1="444.5" y1="175.26" x2="454.66" y2="175.26" width="0.1524" layer="91"/>
-<wire x1="454.66" y1="172.72" x2="454.66" y2="175.26" width="0.1524" layer="91"/>
-<wire x1="454.66" y1="175.26" x2="464.82" y2="175.26" width="0.1524" layer="91"/>
-<wire x1="464.82" y1="172.72" x2="464.82" y2="175.26" width="0.1524" layer="91"/>
-<wire x1="464.82" y1="175.26" x2="474.98" y2="175.26" width="0.1524" layer="91"/>
-<wire x1="474.98" y1="175.26" x2="474.98" y2="172.72" width="0.1524" layer="91"/>
-<wire x1="474.98" y1="175.26" x2="485.14" y2="175.26" width="0.1524" layer="91"/>
-<wire x1="485.14" y1="175.26" x2="485.14" y2="172.72" width="0.1524" layer="91"/>
-<wire x1="485.14" y1="175.26" x2="495.3" y2="175.26" width="0.1524" layer="91"/>
-<wire x1="495.3" y1="175.26" x2="495.3" y2="172.72" width="0.1524" layer="91"/>
-<junction x="454.66" y="175.26"/>
-<junction x="464.82" y="175.26"/>
-<junction x="444.5" y="175.26"/>
-<junction x="474.98" y="175.26"/>
-<pinref part="P+9" gate="G$1" pin="3.3V"/>
-<pinref part="R26" gate="G$1" pin="2"/>
-<pinref part="R27" gate="G$1" pin="2"/>
-<pinref part="R28" gate="G$1" pin="2"/>
-<pinref part="R29" gate="G$1" pin="2"/>
-</segment>
-</net>
 <net name="SDA" class="0">
 <segment>
@@
 </segment>
 <segment>
-<wire x1="485.14" y1="162.56" x2="485.14" y2="121.92" width="0.1524" layer="91"/>
-<wire x1="485.14" y1="121.92" x2="424.18" y2="121.92" width="0.1524" layer="91"/>
-<label x="426.72" y="121.92" size="1.778" layer="95" font="vector"/>
+<wire x1="441.96" y1="226.06" x2="444.5" y2="226.06" width="0.1524" layer="91"/>
 <pinref part="R28" gate="G$1" pin="1"/>
 </segment>
@@
 </segment>
 <segment>
-<wire x1="495.3" y1="162.56" x2="495.3" y2="124.46" width="0.1524" layer="91"/>
-<wire x1="495.3" y1="124.46" x2="424.18" y2="124.46" width="0.1524" layer="91"/>
-<label x="426.72" y="124.46" size="1.778" layer="95" font="vector"/>
+<wire x1="441.96" y1="223.52" x2="444.5" y2="223.52" width="0.1524" layer="91"/>
 <pinref part="R29" gate="G$1" pin="1"/>
 </segment>
@@
 </segment>
 <segment>
-<wire x1="424.18" y1="149.86" x2="474.98" y2="149.86" width="0.1524" layer="91"/>
-<wire x1="474.98" y1="149.86" x2="474.98" y2="162.56" width="0.1524" layer="91"/>
-<label x="426.72" y="149.86" size="1.778" layer="95" font="vector"/>
+<wire x1="444.5" y1="220.98" x2="441.96" y2="220.98" width="0.1524" layer="91"/>
 <pinref part="R27" gate="G$1" pin="1"/>
 </segment>
@@
 </segment>
 <segment>
-<wire x1="424.18" y1="152.4" x2="464.82" y2="152.4" width="0.1524" layer="91"/>
-<wire x1="464.82" y1="152.4" x2="464.82" y2="162.56" width="0.1524" layer="91"/>
-<label x="426.72" y="152.4" size="1.778" layer="95" font="vector"/>
-<pinref part="R26" gate="G$1" pin="1"/>
-</segment>
-</net>
+<pinref part="IC3" gate="G$1" pin="PC0"/>
+<wire x1="63.5" y1="58.42" x2="53.34" y2="58.42" width="0.1524" layer="91"/>
+<label x="53.34" y="58.42" size="1.778" layer="95"/>
+</segment>
+</net>

Commit message: routing
Connections:
- removed net N$21: X1_3.1
Other:
- note added: "Battery Connector"
- moved on the sheet: R27, R28, R29, U1, X1_1, X1_2, X1_3

Commit message: routing
Parts:
- removed U$2: RECEPTABLE_1X4_HORIZ_SMT, seb:RECEPTABLE_1X4_HORIZ_SMT
- added PAD1, PAD2: (no value), wirepad:SMD2
Connections:
- removed net +3V3: C11.2, C12.2, C27.2, C36.2, C37.1, C38.1, C39.1, FERRITE.1, IC3.PA10, IC3.VDD@19, IC3.VDD@32, IC3.VDD@48, IC3.VDD@64, J2-13.MS, J2-14.MS, J2-27.MS, J2-4.MS, L5.2, R27.2, R28.2, R29.2, R32.2, R4.2, SD1.VCC, U1.VDD, U1.VDDP
- new net 3.3V: C11.2, C12.2, C27.2, C36.2, C37.1, C38.1, C39.1, FERRITE.1, IC3.PA10, IC3.VDD@19, IC3.VDD@32, IC3.VDD@48, IC3.VDD@64, J2-13.MS, J2-14.MS, J2-27.MS, J2-4.MS, L5.2, R27.2, R28.2, R29.2, R32.2, R4.2, SD1.VCC, U$1.4, U$1.4@1, U1.VDD, U1.VDDP
- new net N$21: IC3.PC14, PAD1.P
- new net N$23: IC3.PC15, PAD2.P
- net GND: now also U$1.1, U$1.1@1
- net SCL: now also U$1.3, U$1.3@1
- net SDA: now also U$1.2, U$1.2@1
Other:
- moved on the sheet: U$1
Changed lines of the file:
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@@
 <part name="P+2" library="supply1" deviceset="+5V" device=""/>
 <part name="U$1" library="seb" deviceset="RECEPTABLE_1X4_HORIZ_SMT" device=""/>
-<part name="U$2" library="seb" deviceset="RECEPTABLE_1X4_HORIZ_SMT" device=""/>
 <part name="P+1" library="supply1" deviceset="+5V" device=""/>
 <part name="+3V1" library="supply1" deviceset="+3V3" device=""/>
@@
 <part name="GND31" library="supply1" deviceset="GND" device=""/>
 <part name="+3V2" library="supply1" deviceset="+3V3" device=""/>
+<part name="GND32" library="SparkFun" deviceset="GND" device=""/>
+<part name="P+3" library="SparkFun" deviceset="3.3V" device=""/>
+<part name="PAD1" library="wirepad" deviceset="SMD2" device=""/>
+<part name="PAD2" library="wirepad" deviceset="SMD2" device=""/>
 </parts>
 <sheets>
@@
 <instance part="P+4" gate="G$1" x="368.3" y="241.3"/>
 <instance part="P+2" gate="1" x="233.68" y="254"/>
-<instance part="U$1" gate="G$1" x="157.48" y="-68.58"/>
-<instance part="U$2" gate="G$1" x="203.2" y="-68.58"/>
+<instance part="U$1" gate="G$1" x="353.06" y="81.28"/>
 <instance part="P+1" gate="1" x="175.26" y="60.96" rot="R270"/>
 <instance part="+3V1" gate="G$1" x="137.16" y="63.5" rot="R270"/>
@@
 <instance part="GND31" gate="1" x="43.18" y="35.56"/>
 <instance part="+3V2" gate="G$1" x="30.48" y="45.72" rot="R90"/>
+<instance part="GND32" gate="1" x="340.36" y="86.36" rot="R270"/>
+<instance part="P+3" gate="G$1" x="342.9" y="78.74" rot="R90"/>
+<instance part="PAD1" gate="1" x="60.96" y="71.12"/>
+<instance part="PAD2" gate="1" x="60.96" y="68.58"/>
 </instances>
 <busses>
@@
 <pinref part="GND31" gate="1" pin="GND"/>
 </segment>
+<segment>
+<pinref part="U$1" gate="G$1" pin="1"/>
+<pinref part="GND32" gate="1" pin="GND"/>
+<wire x1="342.9" y1="86.36" x2="353.06" y2="86.36" width="0.1524" layer="91"/>
+<pinref part="U$1" gate="G$1" pin="1@1"/>
+<junction x="353.06" y="86.36"/>
+</segment>
 </net>
 <net name="+5V" class="1">
@@
 </segment>
 </net>
-<net name="+3V3" class="2">
+<net name="3.3V" class="2">
 <segment>
 <wire x1="185.42" y1="93.98" x2="185.42" y2="109.22" width="0.1524" layer="91"/>
@@
 <pinref part="+3V2" gate="G$1" pin="+3V3"/>
 </segment>
+<segment>
+<pinref part="P+3" gate="G$1" pin="3.3V"/>
+<pinref part="U$1" gate="G$1" pin="4"/>
+<wire x1="342.9" y1="78.74" x2="353.06" y2="78.74" width="0.1524" layer="91"/>
+<pinref part="U$1" gate="G$1" pin="4@1"/>
+<junction x="353.06" y="78.74"/>
+</segment>
 </net>
 <net name="D-" class="0">
@@
 <net name="N$1" class="0">
 <segment>
-<wire x1="53.34" y1="68.58" x2="60.96" y2="68.58" width="0.1524" layer="91"/>
-<wire x1="60.96" y1="68.58" x2="60.96" y2="66.04" width="0.1524" layer="91"/>
-<wire x1="60.96" y1="66.04" x2="63.5" y2="66.04" width="0.1524" layer="91"/>
+<wire x1="53.34" y1="68.58" x2="55.88" y2="68.58" width="0.1524" layer="91"/>
+<wire x1="55.88" y1="68.58" x2="55.88" y2="66.04" width="0.1524" layer="91"/>
+<wire x1="55.88" y1="66.04" x2="63.5" y2="66.04" width="0.1524" layer="91"/>
 <wire x1="43.18" y1="68.58" x2="53.34" y2="68.58" width="0.1524" layer="91"/>
 <junction x="53.34" y="68.58"/>
@@
 <wire x1="332.74" y1="142.24" x2="335.28" y2="142.24" width="0.1524" layer="91"/>
 <pinref part="R28" gate="G$1" pin="1"/>
+<wire x1="342.9" y1="83.82" x2="353.06" y2="83.82" width="0.1524" layer="91"/>
+<pinref part="U$1" gate="G$1" pin="2"/>
+<pinref part="U$1" gate="G$1" pin="2@1"/>
+<junction x="353.06" y="83.82"/>
+<label x="342.9" y="83.82" size="1.778" layer="95"/>
 </segment>
 <segment>
@@
 <label x="335.28" y="139.7" size="1.778" layer="95"/>
 <pinref part="U1" gate="G$1" pin="SCL"/>
+<wire x1="342.9" y1="81.28" x2="353.06" y2="81.28" width="0.1524" layer="91"/>
+<pinref part="U$1" gate="G$1" pin="3"/>
+<pinref part="U$1" gate="G$1" pin="3@1"/>
+<junction x="353.06" y="81.28"/>
+<label x="342.9" y="81.28" size="1.778" layer="95"/>
 </segment>
 <segment>
@@
 </segment>
 </net>
+<net name="N$21" class="0">
+<segment>
+<pinref part="IC3" gate="G$1" pin="PC14"/>
+<pinref part="PAD1" gate="1" pin="P"/>
+</segment>
+</net>
+<net name="N$23" class="0">
+<segment>
+<pinref part="IC3" gate="G$1" pin="PC15"/>
+<pinref part="PAD2" gate="1" pin="P"/>
+</segment>
+</net>
