File: eagle/lun1k.sch (EAGLE design)
At the start: 105 parts, among them IC1 LTC3558, IC2 LM27313, IC3 STM32F405RGT, IC4 NRF24L01SMD, J2 XF2-3015-1LW, Q1 Q12M-SMD-S, Q2 3.2X2.5CRYSTAL, SW1 JS102011SAQN, SW2 SWITCH_MCTAEF, SW3 SWITCH_MCTAEF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

Commit message: updates
Parts:
- removed C11: 220pF, SparkFun:CAP0805
- removed C12, C33: 1µF, SparkFun:CAP0805
- removed C31, C32: 10µF, rcl:CPOL-EUSMCA
- removed D1: B140F, diode:DIODE-DO214AC
- removed IC2: LM27313, seb:LM27313
- removed L5: 10µH, resistor:L-EUL1812
- removed R11: 15k, rcl:R-EU_R0402
- removed R13: 10k, SparkFun:RESISTOR0805-RES
- removed R5: 100k, SparkFun:RESISTOR0805-RES
- R19: value 1k -> 2.2k
- R8: value 130k -> 150k
- R9: value 680k -> 470k
Connections:
- removed net N$24: D1.A, IC2.SW, L5.2
- removed net N$26: C11.2, IC2.FB, R13.2, R5.1
- net +12V: no longer C11.1, C12.1, D1.C, R5.2
- net 3.3V: no longer C31.+, C32.+, C33.1, IC2.IN, L5.1, R11.2
- net GND: no longer C12.2, C31.-, C32.-, C33.2, IC2.GND, R13.1
- net REG_EN_: no longer IC2./SHDN, R11.1
Changed lines of the file:
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@@
 <?xml version="1.0" encoding="utf-8"?>
 <!DOCTYPE eagle SYSTEM "eagle.dtd">
-<eagle version="6.2">
+<eagle version="6.3">
 <drawing>
 <settings>
@@
 <part name="C7" library="SparkFun" deviceset="CAP" device="0805" value="10pF"/>
 <part name="C8" library="SparkFun" deviceset="CAP" device="0805" value="1µF"/>
-<part name="R8" library="SparkFun-Resistors" deviceset="RESISTOR" device="0805-RES" value="130k"/>
-<part name="R9" library="SparkFun-Resistors" deviceset="RESISTOR" device="0805-RES" value="680k"/>
+<part name="R8" library="SparkFun-Resistors" deviceset="RESISTOR" device="0805-RES" value="150k"/>
+<part name="R9" library="SparkFun-Resistors" deviceset="RESISTOR" device="0805-RES" value="470k"/>
 <part name="R12" library="SparkFun-Resistors" deviceset="RESISTOR" device="0805-RES" value="15k"/>
 <part name="R18" library="SparkFun-Resistors" deviceset="RESISTOR" device="0805-RES" value="121k"/>
-<part name="R19" library="SparkFun-Resistors" deviceset="RESISTOR" device="0805-RES" value="1k"/>
+<part name="R19" library="SparkFun-Resistors" deviceset="RESISTOR" device="0805-RES" value="2.2k"/>
 <part name="GND7" library="supply1" deviceset="GND" device=""/>
 <part name="L1" library="seb" deviceset="SMD-INDUCTOR-4012" device="" value="2,2µH"/>
@@
 <part name="PAD1" library="wirepad" deviceset="SMD2" device=""/>
 <part name="PAD2" library="wirepad" deviceset="SMD2" device=""/>
-<part name="D1" library="diode" deviceset="DIODE-" device="DO214AC" value="B140F"/>
-<part name="L5" library="resistor" deviceset="L-EU" device="L1812" value="10µH"/>
-<part name="IC2" library="seb" deviceset="LM27313" device=""/>
-<part name="R5" library="SparkFun" deviceset="RESISTOR" device="0805-RES" value="100k"/>
-<part name="R13" library="SparkFun" deviceset="RESISTOR" device="0805-RES" value="10k"/>
-<part name="C11" library="SparkFun" deviceset="CAP" device="0805" value="220pF"/>
-<part name="C12" library="SparkFun" deviceset="CAP" device="0805" value="1µF"/>
-<part name="GND33" library="supply1" deviceset="GND" device=""/>
-<part name="+3V6" library="supply1" deviceset="+3V3" device=""/>
-<part name="C31" library="rcl" deviceset="CPOL-EU" device="SMCA" value="10µF"/>
-<part name="C32" library="rcl" deviceset="CPOL-EU" device="SMCA" value="10µF"/>
-<part name="C33" library="SparkFun" deviceset="CAP" device="0805" value="1µF"/>
-<part name="R11" library="rcl" deviceset="R-EU_" device="R0402" value="15k"/>
 <part name="R20" library="SparkFun-Resistors" deviceset="RESISTOR" device="0402-RES" value="680k"/>
 <part name="U$2" library="seb" deviceset="RECEPTABLE_1X4_HORIZ_SMT" device=""/>
@@
 <instance part="PAD1" gate="1" x="58.42" y="71.12"/>
 <instance part="PAD2" gate="1" x="58.42" y="68.58"/>
-<instance part="D1" gate="G$1" x="233.68" y="-25.4"/>
-<instance part="L5" gate="G$1" x="210.82" y="-25.4" rot="R90"/>
-<instance part="IC2" gate="G$1" x="210.82" y="-40.64"/>
-<instance part="R5" gate="G$1" x="243.84" y="-35.56" rot="R90"/>
-<instance part="R13" gate="G$1" x="243.84" y="-50.8" rot="R90"/>
-<instance part="C11" gate="G$1" x="251.46" y="-35.56"/>
-<instance part="C12" gate="G$1" x="261.62" y="-53.34"/>
-<instance part="GND33" gate="1" x="210.82" y="-63.5"/>
-<instance part="+3V6" gate="G$1" x="175.26" y="-22.86"/>
-<instance part="C31" gate="G$1" x="175.26" y="-40.64"/>
-<instance part="C32" gate="G$1" x="165.1" y="-40.64"/>
-<instance part="C33" gate="G$1" x="154.94" y="-43.18"/>
-<instance part="R11" gate="G$1" x="187.96" y="-43.18" rot="R90"/>
 <instance part="R20" gate="G$1" x="53.34" y="63.5" rot="R180"/>
 <instance part="U$2" gate="G$1" x="353.06" y="60.96"/>
@@
 <junction x="353.06" y="86.36"/>
 </segment>
-<segment>
-<wire x1="210.82" y1="-53.34" x2="210.82" y2="-60.96" width="0.1524" layer="91"/>
-<wire x1="210.82" y1="-60.96" x2="243.84" y2="-60.96" width="0.1524" layer="91"/>
-<wire x1="243.84" y1="-60.96" x2="261.62" y2="-60.96" width="0.1524" layer="91"/>
-<wire x1="261.62" y1="-60.96" x2="261.62" y2="-55.88" width="0.1524" layer="91"/>
-<wire x1="210.82" y1="-60.96" x2="193.04" y2="-60.96" width="0.1524" layer="91"/>
-<wire x1="193.04" y1="-60.96" x2="175.26" y2="-60.96" width="0.1524" layer="91"/>
-<wire x1="175.26" y1="-60.96" x2="175.26" y2="-45.72" width="0.1524" layer="91"/>
-<wire x1="243.84" y1="-55.88" x2="243.84" y2="-60.96" width="0.1524" layer="91"/>
-<wire x1="165.1" y1="-45.72" x2="175.26" y2="-45.72" width="0.1524" layer="91"/>
-<wire x1="154.94" y1="-45.72" x2="165.1" y2="-45.72" width="0.1524" layer="91"/>
-<junction x="210.82" y="-60.96"/>
-<junction x="243.84" y="-60.96"/>
-<junction x="175.26" y="-45.72"/>
-<junction x="165.1" y="-45.72"/>
-<pinref part="IC2" gate="G$1" pin="GND"/>
-<pinref part="R13" gate="G$1" pin="1"/>
-<pinref part="C12" gate="G$1" pin="2"/>
-<pinref part="GND33" gate="1" pin="GND"/>
-<pinref part="C31" gate="G$1" pin="-"/>
-<pinref part="C32" gate="G$1" pin="-"/>
-<pinref part="C33" gate="G$1" pin="2"/>
-</segment>
 </net>
 <net name="+5V" class="1">
@@
 <pinref part="R18" gate="G$1" pin="2"/>
 <label x="327.66" y="208.28" size="1.778" layer="95"/>
-</segment>
-<segment>
-<wire x1="193.04" y1="-38.1" x2="187.96" y2="-38.1" width="0.1524" layer="91"/>
-<wire x1="187.96" y1="-38.1" x2="187.96" y2="-25.4" width="0.1524" layer="91"/>
-<wire x1="187.96" y1="-25.4" x2="205.74" y2="-25.4" width="0.1524" layer="91"/>
-<wire x1="187.96" y1="-25.4" x2="175.26" y2="-25.4" width="0.1524" layer="91"/>
-<wire x1="175.26" y1="-25.4" x2="175.26" y2="-38.1" width="0.1524" layer="91"/>
-<wire x1="165.1" y1="-38.1" x2="175.26" y2="-38.1" width="0.1524" layer="91"/>
-<wire x1="154.94" y1="-38.1" x2="165.1" y2="-38.1" width="0.1524" layer="91"/>
-<junction x="187.96" y="-25.4"/>
-<junction x="175.26" y="-25.4"/>
-<junction x="175.26" y="-38.1"/>
-<junction x="165.1" y="-38.1"/>
-<junction x="187.96" y="-38.1"/>
-<pinref part="IC2" gate="G$1" pin="IN"/>
-<pinref part="L5" gate="G$1" pin="1"/>
-<pinref part="+3V6" gate="G$1" pin="+3V3"/>
-<pinref part="C31" gate="G$1" pin="+"/>
-<pinref part="C32" gate="G$1" pin="+"/>
-<pinref part="C33" gate="G$1" pin="1"/>
-<pinref part="R11" gate="G$1" pin="2"/>
 </segment>
 <segment>
@@
 <pinref part="J2" gate="-29" pin="MS"/>
 </segment>
-<segment>
-<wire x1="236.22" y1="-25.4" x2="243.84" y2="-25.4" width="0.1524" layer="91"/>
-<wire x1="243.84" y1="-25.4" x2="251.46" y2="-25.4" width="0.1524" layer="91"/>
-<wire x1="251.46" y1="-25.4" x2="261.62" y2="-25.4" width="0.1524" layer="91"/>
-<wire x1="261.62" y1="-25.4" x2="261.62" y2="-22.86" width="0.1524" layer="91"/>
-<wire x1="261.62" y1="-22.86" x2="269.24" y2="-22.86" width="0.1524" layer="91"/>
-<wire x1="261.62" y1="-25.4" x2="261.62" y2="-48.26" width="0.1524" layer="91"/>
-<wire x1="251.46" y1="-25.4" x2="251.46" y2="-30.48" width="0.1524" layer="91"/>
-<wire x1="243.84" y1="-30.48" x2="243.84" y2="-25.4" width="0.1524" layer="91"/>
-<junction x="261.62" y="-25.4"/>
-<junction x="251.46" y="-25.4"/>
-<junction x="243.84" y="-25.4"/>
-<label x="264.16" y="-22.86" size="1.778" layer="95"/>
-<pinref part="D1" gate="G$1" pin="C"/>
-<pinref part="R5" gate="G$1" pin="2"/>
-<pinref part="C11" gate="G$1" pin="1"/>
-<pinref part="C12" gate="G$1" pin="1"/>
-</segment>
 </net>
 <net name="N$14" class="0">
@@
 </segment>
 </net>
-<net name="N$24" class="0">
-<segment>
-<wire x1="215.9" y1="-25.4" x2="228.6" y2="-25.4" width="0.1524" layer="91"/>
-<wire x1="228.6" y1="-25.4" x2="231.14" y2="-25.4" width="0.1524" layer="91"/>
-<wire x1="228.6" y1="-25.4" x2="228.6" y2="-38.1" width="0.1524" layer="91"/>
-<junction x="228.6" y="-25.4"/>
-<pinref part="L5" gate="G$1" pin="2"/>
-<pinref part="D1" gate="G$1" pin="A"/>
-<pinref part="IC2" gate="G$1" pin="SW"/>
-</segment>
-</net>
-<net name="N$26" class="0">
-<segment>
-<wire x1="228.6" y1="-43.18" x2="243.84" y2="-43.18" width="0.1524" layer="91"/>
-<wire x1="243.84" y1="-43.18" x2="251.46" y2="-43.18" width="0.1524" layer="91"/>
-<wire x1="251.46" y1="-43.18" x2="251.46" y2="-38.1" width="0.1524" layer="91"/>
-<wire x1="243.84" y1="-43.18" x2="243.84" y2="-40.64" width="0.1524" layer="91"/>
-<wire x1="243.84" y1="-43.18" x2="243.84" y2="-45.72" width="0.1524" layer="91"/>
-<junction x="243.84" y="-43.18"/>
-<pinref part="IC2" gate="G$1" pin="FB"/>
-<pinref part="R5" gate="G$1" pin="1"/>
-<pinref part="R13" gate="G$1" pin="2"/>
-<pinref part="C11" gate="G$1" pin="2"/>
-</segment>
-</net>
 <net name="REG_EN_" class="0">
 <segment>
-<wire x1="187.96" y1="-48.26" x2="193.04" y2="-43.18" width="0.1524" layer="91"/>
-<pinref part="IC2" gate="G$1" pin="/SHDN"/>
-<pinref part="R11" gate="G$1" pin="1"/>
-<label x="182.88" y="-50.8" size="1.778" layer="95"/>
-</segment>
-<segment>
 <pinref part="IC3" gate="G$1" pin="PA1"/>
