File: eagle/lun1k.brd (EAGLE design)
At the start: 127.6 x 60.4 mm, 100 parts, among them IC1 LTC3558, IC3 STM32F405RGT, IC4 NRF24L01SMD, J2 XF2-3015-1LW, Q1 Q12M-SMD-S, Q2 3.2X2.5CRYSTAL, SW1 JS102011SAQN, SW2 SWITCH_MCTAEF, SW3 SWITCH_MCTAEF, SW4 SWITCH_MCTAEF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

Commit message: button text
Parts:
- moved R5 36.5 mm to (14.5, 22.8)
- moved R7 34.4 mm to (17.8, 22.9), turned to 270 degrees
- moved R13 32.1 mm to (16.2, 22.8), turned to 90 degrees
Other:
- board text added: "A"
- board text added: "B"
- board text added: "ESC"
- board text added: "bootloader"
- board text added: "wakeup"
Changed lines of the file:
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@@
 <layer number="131" name="tAdjust" color="7" fill="1" visible="no" active="yes"/>
 <layer number="132" name="bAdjust" color="7" fill="1" visible="no" active="yes"/>
-<layer number="142" name="tBestueckung" color="14" fill="1" visible="no" active="yes"/>
+<layer number="142" name="tBestueckung" color="14" fill="1" visible="yes" active="yes"/>
 <layer number="143" name="bBestueckung" color="14" fill="1" visible="no" active="yes"/>
 <layer number="144" name="Drill_legend" color="7" fill="1" visible="no" active="yes"/>
@@
 <wire x1="73.9" y1="13.34" x2="73.9" y2="-13.34" width="0.254" layer="21"/>
 <wire x1="47" y1="13.34" x2="47" y2="-13.34" width="0.254" layer="21"/>
+<text x="2.6" y="14.6" size="1.778" layer="21" font="vector" rot="SR270">A</text>
+<text x="4.6" y="20.1" size="1.778" layer="21" font="vector" rot="SR270">B</text>
+<text x="7" y="27.6" size="1.778" layer="21" font="vector" rot="SR270">ESC</text>
+<text x="-6.5" y="17.8" size="0.8" layer="21" font="vector" ratio="12" rot="SR180">wakeup</text>
+<text x="-2.8" y="28.6" size="0.8" layer="21" font="vector" ratio="12" rot="SR180">bootloader</text>
 </plain>
 <attributes>
@@
 <attribute name="VALUE" x="-13.535" y="0.695" size="1.27" layer="27"/>
 </element>
-<element name="R5" library="SparkFun-Passives" package="0402-RES" value="22k" x="-13.1" y="-1.1" smashed="yes" rot="R90">
-<attribute name="NAME" x="-14.865" y="-0.165" size="1" layer="25" font="vector" rot="SR270"/>
-<attribute name="VALUE" x="-11.195" y="-1.735" size="1.27" layer="27" rot="R90"/>
+<element name="R5" library="SparkFun-Passives" package="0402-RES" value="22k" x="14.5" y="22.8" smashed="yes" rot="R90">
+<attribute name="NAME" x="12.735" y="23.735" size="1" layer="25" font="vector" rot="SR270"/>
+<attribute name="VALUE" x="16.405" y="22.165" size="1.27" layer="27" rot="R90"/>
 </element>
 <element name="R2" library="SparkFun-Passives" package="0402-RES" value="33" x="30.2" y="16.8" smashed="yes">
@@
 <attribute name="VALUE" x="-11.265" y="6.605" size="1.27" layer="27" rot="R180"/>
 </element>
-<element name="R7" library="SparkFun-Passives" package="0402-RES" value="100k" x="-12.6" y="6.8" smashed="yes" rot="R180">
-<attribute name="NAME" x="-9.935" y="5.965" size="1" layer="25" font="vector" rot="SR90"/>
-<attribute name="VALUE" x="-11.965" y="8.705" size="1.27" layer="27" rot="R180"/>
+<element name="R7" library="SparkFun-Passives" package="0402-RES" value="100k" x="17.8" y="22.9" smashed="yes" rot="R270">
+<attribute name="NAME" x="18.635" y="25.565" size="1" layer="25" font="vector" rot="SR180"/>
+<attribute name="VALUE" x="15.895" y="23.535" size="1.27" layer="27" rot="R270"/>
 </element>
 <element name="SW1" library="badge" package="JS102011SAQN" value="JS102011SAQN" x="35.2681" y="-21.4823" smashed="yes" rot="R345"/>
@@
 </element>
 <element name="R22" library="rcl" package="R0603" value="R1002-1%63" x="78" y="10.8"/>
-<element name="R13" library="SparkFun-Passives" package="0402-RES" value="1M" x="-12.8" y="9.1"/>
+<element name="R13" library="SparkFun-Passives" package="0402-RES" value="1M" x="16.2" y="22.8" rot="R90"/>
 <element name="X1_" library="badge" package="JST-PH3" value="JST-PH3" x="8.3" y="-0.6" smashed="yes" rot="R90"/>
 <element name="ANT" library="badge" package="CHIPANTENNA" value="CHIPANTENNA" x="93.3001" y="0"/>
@@
 <wire x1="22.4144" y1="10.4562" x2="24.675" y2="7.25" width="0" layer="19" extent="1-1"/>
 <wire x1="0.6071" y1="22.9216" x2="10.2432" y2="15.258" width="0" layer="19" extent="1-16"/>
-<wire x1="-13.45" y1="9.1" x2="-22.029696875" y2="22.4974125" width="0" layer="19" extent="1-1"/>
 </signal>
 <signal name="+5V" class="1">
@@
 <contactref element="R4" pad="1"/>
 <wire x1="12.8" y1="3.4" x2="12.8" y2="3.6" width="0.2" layer="1"/>
-<wire x1="-13.1" y1="-0.45" x2="12.8" y2="3.4" width="0" layer="19" extent="1-1"/>
-<wire x1="-13.55" y1="2.6" x2="-13.1" y2="-0.45" width="0" layer="19" extent="1-1"/>
+<wire x1="12.8" y1="3.6" x2="14.5" y2="23.45" width="0" layer="19" extent="1-1"/>
+<wire x1="-13.55" y1="2.6" x2="12.8" y2="3.4" width="0" layer="19" extent="1-1"/>
 </signal>
 <signal name="D-">
@@
 <contactref element="R7" pad="2"/>
 <contactref element="R6" pad="1"/>
-<wire x1="-11.25" y1="4.7" x2="-13.25" y2="6.8" width="0" layer="19" extent="1-1"/>
+<wire x1="-11.25" y1="4.7" x2="17.8" y2="22.25" width="0" layer="19" extent="1-1"/>
 </signal>
 <signal name="VCC_EXP" class="1">
 <contactref element="T5" pad="3"/>
 <contactref element="R13" pad="2"/>
-<wire x1="-12.15" y1="9.1" x2="-9.4" y2="1.7" width="0" layer="19" extent="1-1"/>
+<wire x1="-9.4" y1="1.7" x2="16.2" y2="23.45" width="0" layer="19" extent="1-1"/>
 </signal>
 <signal name="+3V3_EXP" class="1">

Commit message: routing
Parts:
- moved C38 1.86 mm to (21.3, 1.53), turned to 270 degrees
Connections:
- new net D2: J2.19
- new net D3: J2.20
- new net D4: J2.21
- new net D5: J2.22
- new net D6: IC3.35, J2.23
- new net D7: IC3.34, J2.24
- new net D8: IC3.33, J2.25
- new net E: J2.16
- new net R/W: J2.15
- net +3V3: now also J2.13, J2.14
- net EN2: no longer IC3.33
- net GND: no longer J2.13, J2.14, J2.15, J2.16
- net N$23: no longer IC3.34
Routing:
- net D6: track 0.00 -> 7.97 mm
- net D7: track 0.00 -> 5.81 mm
- net D8: track 0.00 -> 2.77 mm
- net +12V: track 23.7 -> 26.3 mm
- net +3V3: track 50.0 -> 50.7 mm
Changed lines of the file:
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@@
 <layer number="110" name="fp0" color="7" fill="1" visible="no" active="yes"/>
 <layer number="111" name="LPC17xx" color="7" fill="1" visible="no" active="yes"/>
-<layer number="112" name="tSilk" color="7" fill="1" visible="yes" active="yes"/>
+<layer number="112" name="tSilk" color="7" fill="1" visible="no" active="yes"/>
 <layer number="116" name="Patch_BOT" color="9" fill="4" visible="no" active="yes"/>
 <layer number="121" name="_tsilk" color="7" fill="1" visible="no" active="yes"/>
@@
 <layer number="131" name="tAdjust" color="7" fill="1" visible="no" active="yes"/>
 <layer number="132" name="bAdjust" color="7" fill="1" visible="no" active="yes"/>
-<layer number="142" name="tBestueckung" color="14" fill="1" visible="yes" active="yes"/>
+<layer number="142" name="tBestueckung" color="14" fill="1" visible="no" active="yes"/>
 <layer number="143" name="bBestueckung" color="14" fill="1" visible="no" active="yes"/>
 <layer number="144" name="Drill_legend" color="7" fill="1" visible="no" active="yes"/>
 <layer number="151" name="HeatSink" color="7" fill="1" visible="no" active="yes"/>
-<layer number="152" name="_bDocu" color="7" fill="1" visible="yes" active="yes"/>
+<layer number="152" name="_bDocu" color="7" fill="1" visible="no" active="yes"/>
 <layer number="199" name="Contour" color="7" fill="1" visible="no" active="yes"/>
 <layer number="200" name="200bmp" color="1" fill="10" visible="no" active="yes"/>
@@
 <element name="C36" library="SparkFun-Capacitors" package="0402-CAP" value="100nF" x="22.409" y="15.003" rot="R270"/>
 <element name="C37" library="SparkFun-Capacitors" package="0402-CAP" value="100nF" x="10.8932" y="15.258" rot="R180"/>
-<element name="C38" library="SparkFun-Capacitors" package="0402-CAP" value="100nF" x="22.0696" y="3.246"/>
+<element name="C38" library="SparkFun-Capacitors" package="0402-CAP" value="100nF" x="21.346" y="1.5304" rot="R270"/>
 <element name="IC3" library="stm32" package="LQFP64" value="STM32F405RGT" x="16.4144" y="9.2062" smashed="yes" rot="R270">
 <attribute name="NAME" x="21.9144" y="16.2062" size="1.016" layer="25" ratio="25" rot="R270"/>
@@
 <wire x1="-12.55" y1="4.7" x2="-7.95" y2="6.3" width="0" layer="19" extent="1-1"/>
 </signal>
-<signal name="GND" class="2">
+<signal name="GND" class="2" airwireshidden="yes">
 <contactref element="X1" pad="GND"/>
 <contactref element="R5" pad="1"/>
@@
 <vertex x="-26.5" y="30"/>
 </polygon>
-<polygon width="0.3" layer="1" isolate="0.3">
+<polygon width="0.3" layer="1" isolate="90.3">
 <vertex x="89" y="30"/>
 <vertex x="89" y="2.1"/>
@@
 <contactref element="C29" pad="-"/>
 <contactref element="D2" pad="3"/>
-<contactref element="J2" pad="13"/>
-<contactref element="J2" pad="14"/>
-<contactref element="J2" pad="15"/>
-<contactref element="J2" pad="16"/>
 <contactref element="J2" pad="12"/>
 <contactref element="C38" pad="2"/>
@@
 <wire x1="16.1644" y1="15.2062" x2="13.1644" y2="15.2062" width="0" layer="19" extent="1-1"/>
 <wire x1="18.6644" y1="15.2062" x2="16.1644" y2="15.2062" width="0" layer="19" extent="1-1"/>
-<wire x1="24.675" y1="0.25" x2="22.7196" y2="3.246" width="0" layer="19" extent="1-1"/>
 <wire x1="17.2" y1="-12.4" x2="18.8" y2="-9.05" width="0" layer="19" extent="1-1"/>
 <wire x1="22.4144" y1="10.4562" x2="24.675" y2="7.25" width="0" layer="19" extent="1-1"/>
+<wire x1="24.675" y1="-1.75" x2="29.1" y2="-1.3" width="0" layer="19" extent="1-1"/>
 <wire x1="0.6071" y1="22.9216" x2="10.2432" y2="15.258" width="0" layer="19" extent="1-16"/>
 </signal>
@@
 <wire x1="13.6646" y1="1.5898" x2="13.6644" y2="1.59" width="0.254" layer="1"/>
 <wire x1="13.6644" y1="1.59" x2="13.6644" y2="3.2062" width="0.254" layer="1"/>
-<wire x1="20.1644" y1="3.2062" x2="20.2042" y2="3.246" width="0.254" layer="1"/>
-<wire x1="20.2042" y1="3.246" x2="21.4196" y2="3.246" width="0.254" layer="1"/>
 <wire x1="22.4144" y1="12.9562" x2="22.4144" y2="14.3476" width="0.254" layer="1"/>
 <wire x1="22.4144" y1="14.3476" x2="22.409" y2="14.353" width="0.254" layer="1"/>
@@
 <wire x1="8" y1="-18.8" x2="8" y2="-0.7" width="0.3048" layer="16"/>
 <wire x1="8" y1="-0.7" x2="13.7" y2="5" width="0.3048" layer="16"/>
+<contactref element="J2" pad="13"/>
+<contactref element="J2" pad="14"/>
 <wire x1="24.675" y1="5.75" x2="70.5" y2="2.7" width="0" layer="19" extent="1-1"/>
-<wire x1="21.4196" y1="3.246" x2="24.675" y2="5.75" width="0" layer="19" extent="1-1"/>
+<wire x1="21.346" y1="2.1804" x2="24.675" y2="5.75" width="0" layer="19" extent="1-1"/>
+<wire x1="24.675" y1="-0.75" x2="21.346" y2="2.1804" width="0" layer="19" extent="1-1"/>
+<wire x1="24.675" y1="-1.25" x2="24.675" y2="-0.75" width="0" layer="19" extent="1-1"/>
+<wire x1="24.675" y1="-5.75" x2="24.675" y2="-1.25" width="0" layer="19" extent="1-1"/>
 <wire x1="13.6644" y1="3.2062" x2="20.1644" y2="3.2062" width="0" layer="19" extent="1-1"/>
 <wire x1="13.7" y1="5" x2="13.6644" y2="3.2062" width="0" layer="19" extent="1-16"/>
 <wire x1="22.4144" y1="12.9562" x2="24.675" y2="5.75" width="0" layer="19" extent="1-1"/>
-<wire x1="24.675" y1="-5.75" x2="21.4196" y2="3.246" width="0" layer="19" extent="1-1"/>
 <wire x1="12.6644" y1="15.2062" x2="22.4144" y2="14.3476" width="0" layer="19" extent="1-1"/>
 <wire x1="-3.519009375" y1="-24.296334375" x2="8" y2="-18.8" width="0" layer="19" extent="1-16"/>
 <wire x1="-3.313796875" y1="-24.86015" x2="-3.519009375" y2="-24.296334375" width="0" layer="19" extent="1-1"/>
 <wire x1="-7" y1="-2.25" x2="8" y2="-0.7" width="0" layer="19" extent="1-16"/>
+<wire x1="20.1644" y1="3.2062" x2="20.9938" y2="3.2062" width="0.254" layer="1"/>
+<wire x1="20.9938" y1="3.2062" x2="21.346" y2="2.854" width="0.254" layer="1"/>
+<wire x1="21.346" y1="2.854" x2="21.346" y2="2.1804" width="0.254" layer="1"/>
 </signal>
 <signal name="USB_VBUS">
@@
 <wire x1="22.7" y1="-19.6" x2="21.5" y2="-19.6" width="0.3048" layer="1"/>
 <wire x1="24.675" y1="6.75" x2="60.78" y2="19.3894" width="0" layer="19" extent="1-1"/>
-<wire x1="24.675" y1="-6.75" x2="24.675" y2="6.75" width="0" layer="19" extent="1-1"/>
+<wire x1="24.675" y1="6.75" x2="27.2" y2="6.75" width="0.254" layer="1"/>
+<wire x1="27.2" y1="6.75" x2="27.2" y2="6.7" width="0.254" layer="1"/>
+<wire x1="27.2" y1="6.7" x2="24.675" y2="-6.75" width="0" layer="19" extent="1-16"/>
 </signal>
 <signal name="N$14">
@@
 <signal name="N$23">
 <contactref element="IC1" pad="19"/>
-<contactref element="IC3" pad="34"/>
 <wire x1="15.9" y1="-13.6" x2="15.9" y2="-12.2" width="0.2032" layer="1"/>
 <wire x1="15.9" y1="-12.2" x2="15.4" y2="-11.7" width="0.2032" layer="1"/>
 <via x="15.4" y="-11.7" extent="1-16" drill="0.4"/>
 <wire x1="15.4" y1="-11.7" x2="15.4" y2="-7.2" width="0.2032" layer="16"/>
-<wire x1="15.4" y1="-7.2" x2="22.4144" y2="5.9562" width="0" layer="19" extent="1-16"/>
 </signal>
 <signal name="EN2">
 <contactref element="IC1" pad="15"/>
 <contactref element="R24" pad="2"/>
-<contactref element="IC3" pad="33"/>
 <wire x1="17.7" y1="-14.2" x2="17.7" y2="-14" width="0.2032" layer="1"/>
 <wire x1="17.7" y1="-14" x2="18.7" y2="-13" width="0.2032" layer="1"/>
 <wire x1="18.7" y1="-13" x2="18.7" y2="-10.45" width="0.2032" layer="1"/>
 <wire x1="18.7" y1="-10.45" x2="18.8" y2="-10.35" width="0.2032" layer="1"/>
-<wire x1="18.8" y1="-10.35" x2="22.4144" y2="5.4562" width="0" layer="19" extent="1-1"/>
 </signal>
 <signal name="N$25">
@@
 <wire x1="15" y1="-16.8" x2="12.7" y2="-16.8" width="0.3048" layer="1"/>
 </signal>
+<signal name="D2">
+<contactref element="J2" pad="19"/>
+</signal>
+<signal name="D3">
+<contactref element="J2" pad="20"/>
+</signal>
+<signal name="D4">
+<contactref element="J2" pad="21"/>
+</signal>
+<signal name="D5">
+<contactref element="J2" pad="22"/>
+</signal>
+<signal name="D6">
+<contactref element="J2" pad="23"/>
+<contactref element="IC3" pad="35"/>
+<wire x1="24.675" y1="3.75" x2="21.35" y2="3.75" width="0.254" layer="1"/>
+<wire x1="21.35" y1="3.75" x2="20.5" y2="4.6" width="0.254" layer="1"/>
+<wire x1="20.5" y1="4.6" x2="20.5" y2="5.9" width="0.254" layer="1"/>
+<wire x1="20.5" y1="5.9" x2="21.0562" y2="6.4562" width="0.254" layer="1"/>
+<wire x1="21.0562" y1="6.4562" x2="22.4144" y2="6.4562" width="0.254" layer="1"/>
+</signal>
+<signal name="D7">
+<contactref element="J2" pad="24"/>
+<contactref element="IC3" pad="34"/>
+<wire x1="24.675" y1="4.25" x2="21.85" y2="4.25" width="0.254" layer="1"/>
+<wire x1="21.85" y1="4.25" x2="21.2" y2="4.9" width="0.254" layer="1"/>
+<wire x1="21.2" y1="4.9" x2="21.2" y2="5.6" width="0.254" layer="1"/>
+<wire x1="21.2" y1="5.6" x2="21.5562" y2="5.9562" width="0.254" layer="1"/>
+<wire x1="21.5562" y1="5.9562" x2="22.4144" y2="5.9562" width="0.254" layer="1"/>
+</signal>
+<signal name="D8">
+<contactref element="J2" pad="25"/>
+<contactref element="IC3" pad="33"/>
+<wire x1="24.675" y1="4.75" x2="22.75" y2="4.75" width="0.254" layer="1"/>
+<wire x1="22.75" y1="4.75" x2="22.4144" y2="5.0856" width="0.254" layer="1"/>
+<wire x1="22.4144" y1="5.0856" x2="22.4144" y2="5.4562" width="0.254" layer="1"/>
+</signal>
+<signal name="R/W" class="2">
+<contactref element="J2" pad="15"/>
+</signal>
+<signal name="E" class="2">
+<contactref element="J2" pad="16"/>
+</signal>
 </signals>

Commit message: routing
Parts:
- moved C40 1.30 mm to (19.8, 0.33), turned to 270 degrees
Connections:
- net D/C: now also IC3.25
- net D0: now also IC3.29
- net D1: now also IC3.30
- net D2: now also IC3.40
- net D3: now also IC3.39
- net D4: now also IC3.38
- net D5: now also IC3.36
- net E: now also IC3.27
- net GND: no longer IC3.30
- net R/W: now also IC3.26
- net RES: now also IC3.24
Routing:
- net D/C: track 0.00 -> 21.2 mm, vias 0 -> 2
- net E: track 0.00 -> 19.7 mm, vias 0 -> 2
- net R/W: track 0.00 -> 16.5 mm, vias 0 -> 2
- net RES: track 0.00 -> 15.9 mm, vias 0 -> 2
- net D2: track 0.00 -> 15.2 mm, vias 0 -> 2
- net D1: track 0.00 -> 14.5 mm, vias 0 -> 2
- net D3: track 0.00 -> 12.8 mm, vias 0 -> 2
- net D5: track 0.00 -> 11.4 mm, vias 0 -> 2
- net D4: track 0.00 -> 11.4 mm, vias 0 -> 2
- net D0: track 0.00 -> 9.79 mm, vias 0 -> 2

Commit message: routeing
Connections:
- net D0: now also IC3.26; no longer IC3.29
- net D1: now also IC3.27; no longer IC3.30
- net D2: now also IC3.29; no longer IC3.40
- net D3: now also IC3.30; no longer IC3.39
- net D4: now also IC3.36; no longer IC3.38
- net D5: now also IC3.35; no longer IC3.36
- net D6: now also IC3.34; no longer IC3.35
- net D7: now also IC3.33; no longer IC3.34
- net D8: no longer IC3.33
- net E: now also IC3.38; no longer IC3.27
- net R/W: now also IC3.40; no longer IC3.26
Routing:
- net D2: track 15.2 -> 8.49 mm
- net R/W: track 16.5 -> 22.1 mm
- net D/C: track 21.2 -> 17.5 mm
- net E: track 19.7 -> 16.3 mm
- net D1: track 14.5 -> 17.4 mm
- net D8: track 2.77 -> 0.00 mm
- net D7: track 5.81 -> 3.15 mm
- net D6: track 7.97 -> 6.47 mm
- net D0: track 9.79 -> 11.3 mm

Commit message: routing
Parts:
- moved F1 35.6 mm to (35.4, -13.0)
- moved C1 1.30 mm to (10.8, -10.8)
- moved R19 0.70 mm to (16.7, -9.40)
- moved C8 0.30 mm to (13.7, -9.40)
Connections:
- new net N$8: F1.1, X1.VUSB
- net +5V: now also F1.2; no longer X1.VUSB
- net VCC: no longer F1.2
Routing:
- net +5V: track 75.6 -> 38.9 mm
- net N$8: track 0.00 -> 34.9 mm
- net N$23: track 6.61 -> 3.49 mm, vias 1 -> 0
