File: eagle/lun1k.brd (EAGLE design)
At the start: 127.6 x 60.4 mm, 102 parts, among them IC1 LTC3558, IC3 STM32F405RGT, IC4 NRF24L01SMD, J2 XF2-3015-1LW, Q1 Q12M-SMD-S, Q2 3.2X2.5CRYSTAL, SW1 JS102011SAQN, SW2 SWITCH_MCTAEF, SW3 SWITCH_MCTAEF, SW4 SWITCH_MCTAEF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

Commit message: routing
Parts:
- removed R11, R4: 10k, SparkFun-Passives:0402-RES
- removed R13: 1M, SparkFun-Passives:0402-RES
- removed R5: 22k, SparkFun-Passives:0402-RES
- removed T5, T6: SI2301DS, transistor-small-signal:SOT23
- moved C29 5.32 mm to (27.0, 17.4)
- moved C28 5.10 mm to (29.0, 17.1)
- moved R2 4.87 mm to (34.8, 15.2)
- moved R3 1.77 mm to (34.8, 13.6)
Connections:
- removed net +3V3_EXP: C27.2, SD1.4, T6.3
- removed net POWER_GOOD: R11.1, T5.1, T6.1
- removed net USB_VBUS: R4.1, R5.2
- removed net VCC_EXP: R13.2, T5.3
- net +3V3: now also C27.2, IC3.43, SD1.4; no longer T6.2
- net +5V: now also IC3.42; no longer R4.2
- net GND: no longer IC3.43, R13.1, R5.1
- net USB_DM: now also IC3.44
- net USB_DP: now also IC3.45
- net VCC: no longer R11.2, T5.2
Routing:
- net USB_DP: track 0.00 -> 13.3 mm
- net USB_DM: track 0.00 -> 12.8 mm
- net D+: track 0.57 -> 3.21 mm
- net GND: vias 67 -> 66

Commit message: routing
Parts:
- removed R20: 10k, SparkFun:0402-RES
- removed SJ1: SOLDERJUMPERNO, SparkFun:SJ_2S-NO
- moved R7 36.7 mm to (-12.3, 1.90), turned to 0 degrees
- moved R29 13.4 mm to (-10.1, -23.6), turned to 180 degrees
- moved R28 13.3 mm to (-10.1, -25.0), turned to 180 degrees
- moved R27 12.8 mm to (-10.1, -22.2), turned to 180 degrees
- moved R21 11.6 mm to (-10.1, -19.3), turned to 180 degrees
- moved R26 10.2 mm to (-10.1, -20.8), turned to 180 degrees
- moved R6 4.74 mm to (-12.5, 0.00)
Connections:
- removed net ADDR: R20.1, SJ1.2, U1.9
- net 3.3V: no longer R20.2
- net GND: now also U1.9; no longer SJ1.1
Routing:
- net SDA: track 0.00 -> 6.09 mm
- net SWITCHN: track 0.00 -> 6.01 mm
- net SCL: track 0.00 -> 5.56 mm
- net INTN: track 0.00 -> 5.56 mm
- net RESETN: track 0.00 -> 5.44 mm
Changed lines of the file:
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@@
 <attribute name="VALUE" x="-17.365" y="27.905" size="1.27" layer="27" rot="R180"/>
 </element>
-<element name="R6" library="SparkFun-Passives" package="0402-RES" value="220k" x="-11.9" y="4.7" smashed="yes" rot="R180">
-<attribute name="NAME" x="-14.565" y="5.435" size="1" layer="25" font="vector" rot="SR270"/>
-<attribute name="VALUE" x="-11.265" y="6.605" size="1.27" layer="27" rot="R180"/>
-</element>
-<element name="R7" library="SparkFun-Passives" package="0402-RES" value="100k" x="17.8" y="22.9" smashed="yes" rot="R270">
-<attribute name="NAME" x="18.635" y="25.565" size="1" layer="25" font="vector" rot="SR180"/>
-<attribute name="VALUE" x="15.895" y="23.535" size="1.27" layer="27" rot="R270"/>
+<element name="R6" library="SparkFun-Passives" package="0402-RES" value="220k" x="-12.5" y="0" smashed="yes" rot="R180">
+<attribute name="NAME" x="-15.165" y="0.735" size="1" layer="25" font="vector" rot="SR270"/>
+<attribute name="VALUE" x="-11.865" y="1.905" size="1.27" layer="27" rot="R180"/>
+</element>
+<element name="R7" library="SparkFun-Passives" package="0402-RES" value="100k" x="-12.3" y="1.9" smashed="yes">
+<attribute name="NAME" x="-14.965" y="2.735" size="1" layer="25" font="vector" rot="SR270"/>
+<attribute name="VALUE" x="-12.935" y="-0.005" size="1.27" layer="27"/>
 </element>
 <element name="SW1" library="badge" package="JS102011SAQN" value="JS102011SAQN" x="35.2681" y="-21.4823" smashed="yes" rot="R345"/>
@@
 <element name="C41" library="SparkFun" package="0805" value="2,2µF" x="24.6914" y="13.334" rot="R270"/>
 <element name="U1" library="miscellany" package="N35P112" value="N35P112" x="0" y="-21.1" rot="R20"/>
-<element name="R20" library="SparkFun" package="0402-RES" value="10k" x="-18.7" y="-12"/>
-<element name="R21" library="SparkFun" package="0402-RES" value="10k" x="-16.5" y="-9.6"/>
-<element name="R26" library="SparkFun" package="0402-RES" value="10k" x="-15.3" y="-12"/>
-<element name="R27" library="SparkFun" package="0402-RES" value="10k" x="-12.8" y="-9.7"/>
-<element name="SJ1" library="SparkFun" package="SJ_2S-NO" value="SOLDERJUMPERNO" x="-6.6" y="-27.7"/>
-<element name="R28" library="SparkFun" package="0402-RES" value="10k" x="-12" y="-11.8"/>
-<element name="R29" library="SparkFun" package="0402-RES" value="10k" x="-9.6" y="-10.2"/>
+<element name="R21" library="SparkFun" package="0402-RES" value="10k" x="-10.1" y="-19.3" rot="R180"/>
+<element name="R26" library="SparkFun" package="0402-RES" value="10k" x="-10.1" y="-20.8" rot="R180"/>
+<element name="R27" library="SparkFun" package="0402-RES" value="10k" x="-10.1" y="-22.2" rot="R180"/>
+<element name="R28" library="SparkFun" package="0402-RES" value="10k" x="-10.1" y="-25" rot="R180"/>
+<element name="R29" library="SparkFun" package="0402-RES" value="10k" x="-10.1" y="-23.6" rot="R180"/>
 <element name="SW2" library="seb" package="SWITCH_MCTAEF" value="SWITCH_MCTAEF" x="2.1" y="26.8" rot="R340"/>
 <element name="SW3" library="seb" package="SWITCH_MCTAEF" value="SWITCH_MCTAEF" x="0" y="21.2" rot="R340"/>
@@
 <contactref element="U1" pad="11"/>
 <contactref element="U1" pad="10"/>
-<contactref element="SJ1" pad="1"/>
 <contactref element="IC1" pad="1"/>
 <contactref element="IC1" pad="21"/>
@@
 <wire x1="16.7" y1="-14.6" x2="16.3" y2="-15" width="0.2032" layer="1"/>
 <via x="16.3" y="-15" extent="1-16" drill="0.6"/>
+<contactref element="U1" pad="9"/>
 <wire x1="16.1644" y1="15.2062" x2="18.6644" y2="15.2062" width="0" layer="19" extent="1-1"/>
 <wire x1="13.1644" y1="15.2062" x2="16.1644" y2="15.2062" width="0" layer="19" extent="1-1"/>
@@
 <contactref element="R7" pad="2"/>
 <contactref element="R6" pad="1"/>
-<wire x1="-11.25" y1="4.7" x2="17.8" y2="22.25" width="0" layer="19" extent="1-1"/>
+<wire x1="-11.85" y1="0" x2="-11.65" y2="1.9" width="0" layer="19" extent="1-1"/>
 </signal>
 <signal name="SCK">
@@
 </signal>
 <signal name="3.3V">
-<contactref element="R20" pad="2"/>
 <contactref element="R21" pad="2"/>
 <contactref element="R26" pad="2"/>
@@
 <contactref element="R28" pad="2"/>
 <contactref element="R29" pad="2"/>
-<wire x1="-15.85" y1="-9.6" x2="-18.05" y2="-12" width="0" layer="19" extent="1-1"/>
-<wire x1="-14.65" y1="-12" x2="-15.85" y2="-9.6" width="0" layer="19" extent="1-1"/>
-<wire x1="-11.35" y1="-11.8" x2="-14.65" y2="-12" width="0" layer="19" extent="1-1"/>
-<wire x1="-12.15" y1="-9.7" x2="-11.35" y2="-11.8" width="0" layer="19" extent="1-1"/>
-<wire x1="-8.95" y1="-10.2" x2="-11.35" y2="-11.8" width="0" layer="19" extent="1-1"/>
+<wire x1="-10.75" y1="-23.6" x2="-10.75" y2="-25" width="0" layer="19" extent="1-1"/>
+<wire x1="-10.75" y1="-22.2" x2="-10.75" y2="-23.6" width="0" layer="19" extent="1-1"/>
+<wire x1="-10.75" y1="-20.8" x2="-10.75" y2="-22.2" width="0" layer="19" extent="1-1"/>
+<wire x1="-10.75" y1="-19.3" x2="-10.75" y2="-20.8" width="0" layer="19" extent="1-1"/>
 </signal>
 <signal name="SDA">
 <contactref element="U1" pad="4"/>
 <contactref element="R28" pad="1"/>
-<wire x1="-12.65" y1="-11.8" x2="-3.929434375" y2="-23.168703125" width="0" layer="19" extent="1-1"/>
+<wire x1="-3.929434375" y1="-23.168703125" x2="-6.1" y2="-24" width="0.2286" layer="1"/>
+<wire x1="-6.1" y1="-24" x2="-7.1" y2="-25" width="0.2286" layer="1"/>
+<wire x1="-7.1" y1="-25" x2="-9.45" y2="-25" width="0.2286" layer="1"/>
 </signal>
 <signal name="SCL">
 <contactref element="U1" pad="5"/>
 <contactref element="R29" pad="1"/>
-<wire x1="-10.25" y1="-10.2" x2="-4.134646875" y2="-22.6048875" width="0" layer="19" extent="1-1"/>
+<wire x1="-4.134646875" y1="-22.6048875" x2="-6.1" y2="-23.3" width="0.2286" layer="1"/>
+<wire x1="-6.1" y1="-23.3" x2="-7.2" y2="-23.3" width="0.2286" layer="1"/>
+<wire x1="-7.2" y1="-23.3" x2="-7.5" y2="-23.6" width="0.2286" layer="1"/>
+<wire x1="-7.5" y1="-23.6" x2="-9.45" y2="-23.6" width="0.2286" layer="1"/>
 </signal>
 <signal name="RESETN">
 <contactref element="U1" pad="6"/>
 <contactref element="R27" pad="1"/>
-<wire x1="-13.45" y1="-9.7" x2="-4.339859375" y2="-22.041071875" width="0" layer="19" extent="1-1"/>
-</signal>
-<signal name="ADDR">
-<contactref element="U1" pad="9"/>
-<contactref element="R20" pad="1"/>
-<contactref element="SJ1" pad="2"/>
-<wire x1="-4.95549375" y1="-20.349625" x2="-6.15" y2="-27.7" width="0" layer="19" extent="1-1"/>
-<wire x1="-19.35" y1="-12" x2="-4.95549375" y2="-20.349625" width="0" layer="19" extent="1-1"/>
+<wire x1="-4.339859375" y1="-22.041071875" x2="-6.1" y2="-22.7" width="0.2286" layer="1"/>
+<wire x1="-6.1" y1="-22.7" x2="-7.4" y2="-22.7" width="0.2286" layer="1"/>
+<wire x1="-7.4" y1="-22.7" x2="-7.9" y2="-22.2" width="0.2286" layer="1"/>
+<wire x1="-7.9" y1="-22.2" x2="-9.45" y2="-22.2" width="0.2286" layer="1"/>
 </signal>
 <signal name="INTN">
 <contactref element="U1" pad="7"/>
 <contactref element="R26" pad="1"/>
-<wire x1="-4.54506875" y1="-21.47725625" x2="-15.95" y2="-12" width="0" layer="19" extent="1-1"/>
+<wire x1="-4.54506875" y1="-21.47725625" x2="-6.2" y2="-22.1" width="0.2286" layer="1"/>
+<wire x1="-6.2" y1="-22.1" x2="-7.2" y2="-22.1" width="0.2286" layer="1"/>
+<wire x1="-7.2" y1="-22.1" x2="-8.5" y2="-20.8" width="0.2286" layer="1"/>
+<wire x1="-8.5" y1="-20.8" x2="-9.45" y2="-20.8" width="0.2286" layer="1"/>
 </signal>
 <signal name="SWITCHN">
 <contactref element="U1" pad="8"/>
 <contactref element="R21" pad="1"/>
-<wire x1="-17.15" y1="-9.6" x2="-4.75028125" y2="-20.913440625" width="0" layer="19" extent="1-1"/>
+<wire x1="-4.75028125" y1="-20.913440625" x2="-6.4" y2="-21.5" width="0.2286" layer="1"/>
+<wire x1="-6.4" y1="-21.5" x2="-7" y2="-21.5" width="0.2286" layer="1"/>
+<wire x1="-7" y1="-21.5" x2="-8.4" y2="-20.1" width="0.2286" layer="1"/>
+<wire x1="-8.4" y1="-20.1" x2="-8.4" y2="-19.6" width="0.2286" layer="1"/>
+<wire x1="-8.4" y1="-19.6" x2="-8.7" y2="-19.3" width="0.2286" layer="1"/>
+<wire x1="-8.7" y1="-19.3" x2="-9.45" y2="-19.3" width="0.2286" layer="1"/>
 </signal>
 <signal name="N$21" class="1">

Commit message: routing
Parts:
- moved R6 23.3 mm to (10.5, 3.60), turned to 270 degrees
- moved R7 20.6 mm to (8.00, 5.40)
- moved C27 2.71 mm to (12.5, 20.6), flipped to the top
Connections:
- removed net VCC: R6.2
- net GND: no longer IC3.52
- net MISO: now also IC3.52
- net MOSI: now also IC3.53
- net SCK: now also IC3.51
- net VLIPO: now also R6.2
Routing:
- net SCK: track 12.8 -> 96.0 mm, vias 0 -> 2
- net MISO: track 14.9 -> 96.2 mm, vias 0 -> 2
- net MOSI: track 14.5 -> 91.0 mm, vias 0 -> 2
- net GND: track 122.6 -> 58.5 mm
- net CSN: track 42.0 -> 27.9 mm, vias 2 -> 1
- net SS3: track 1.02 -> 0.00 mm

Commit message: routing
Parts:
- moved C27 7.22 mm to (6.70, 16.3), turned to 180 degrees
- moved SW3 0.20 mm to (0.00, 21.0), turned to 160 degrees
- moved SW2 0.10 mm to (2.00, 26.8), turned to 160 degrees
Connections:
- new net SW2: IC3.60, IC3.61, SW2.1
- new net SW3: IC3.59, SW3.1
- new net SW4: IC3.2, SW4.1
- net SS3: now also IC3.62
Routing:
- net SW3: track 0.00 -> 27.1 mm
- net +3V3: track 50.7 -> 76.5 mm, vias 1 -> 2
- net SW2: track 0.00 -> 16.1 mm
- net SS3: track 0.00 -> 14.9 mm, vias 0 -> 1
- net SW4: track 0.00 -> 10.0 mm
Changed lines of the file:
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@@
 <element name="X1_" library="badge" package="JST-PH3" value="JST-PH3" x="8.3" y="-0.6" smashed="yes" rot="R90"/>
 <element name="ANT" library="badge" package="CHIPANTENNA" value="CHIPANTENNA" x="93.3001" y="0"/>
-<element name="C27" library="rcl" package="C0805K" value="10uF" x="12.5" y="20.6" rot="R90"/>
+<element name="C27" library="rcl" package="C0805K" value="10uF" x="6.7" y="16.3" rot="R180"/>
 <element name="R1" library="SparkFun" package="0805" value="1M" x="34.0534" y="-2.265"/>
 <element name="R10" library="SparkFun" package="0805" value="50R" x="34.4838" y="4.335"/>
@@
 <element name="R28" library="SparkFun" package="0402-RES" value="10k" x="-10.1" y="-25" rot="R180"/>
 <element name="R29" library="SparkFun" package="0402-RES" value="10k" x="-10.1" y="-23.6" rot="R180"/>
-<element name="SW2" library="seb" package="SWITCH_MCTAEF" value="SWITCH_MCTAEF" x="2.1" y="26.8" rot="R340"/>
-<element name="SW3" library="seb" package="SWITCH_MCTAEF" value="SWITCH_MCTAEF" x="0" y="21.2" rot="R340"/>
+<element name="SW2" library="seb" package="SWITCH_MCTAEF" value="SWITCH_MCTAEF" x="2" y="26.8" rot="R160"/>
+<element name="SW3" library="seb" package="SWITCH_MCTAEF" value="SWITCH_MCTAEF" x="0" y="21" rot="R160"/>
 <element name="SW4" library="seb" package="SWITCH_MCTAEF" value="SWITCH_MCTAEF" x="-2.1" y="15.5" rot="R160"/>
 <element name="IC1" library="seb" package="UD-QFN20" value="LTC3558" x="16.3" y="-15"/>
@@
 <contactref element="C27" pad="1"/>
 <wire x1="36.3" y1="16" x2="36.4" y2="16.1" width="0.2" layer="16"/>
-<wire x1="41" y1="5.3" x2="36.3" y2="10" width="0" layer="19" extent="1-16"/>
-<wire x1="36.3" y1="10" x2="36.3" y2="16" width="0" layer="19" extent="1-16"/>
 <wire x1="77.2217" y1="4.675" x2="78.6" y2="4.675" width="0.2" layer="1"/>
 <wire x1="78.3892" y1="2.154" x2="78.354" y2="2.154" width="0.2" layer="1"/>
 <wire x1="78.4" y1="2.154" x2="78.3892" y2="2.154" width="0.2" layer="1"/>
 <wire x1="81.4" y1="2" x2="81.4" y2="2.055" width="0.2" layer="16"/>
-<wire x1="41" y1="0.3" x2="41" y2="5.3" width="0" layer="19" extent="1-16"/>
-<wire x1="41" y1="0.3" x2="53.8" y2="0.3" width="0" layer="19" extent="1-16"/>
-<wire x1="53.8" y1="0.3" x2="59" y2="0.3" width="0" layer="19" extent="1-16"/>
-<wire x1="59" y1="0.3" x2="60.5" y2="1.8" width="0" layer="19" extent="1-16"/>
-<wire x1="68.7012" y1="1.7012" x2="68.7012" y2="-4.375" width="0" layer="19" extent="1-16"/>
-<wire x1="68.8" y1="1.8" x2="68.7012" y2="1.7012" width="0" layer="19" extent="1-16"/>
-<wire x1="60.5" y1="1.8" x2="68.8" y2="1.8" width="0" layer="19" extent="1-16"/>
 <wire x1="78.3892" y1="2.154" x2="78.3892" y2="0.9658" width="0.3" layer="1"/>
 <wire x1="78.3892" y1="0.9658" x2="78.58" y2="0.875" width="0.2" layer="1"/>
@@
 <wire x1="78.5065" y1="-0.975" x2="78.5065" y2="-0.8935" width="0.2" layer="1"/>
 <wire x1="78.5065" y1="-0.8935" x2="79.4" y2="0" width="0.2" layer="1"/>
-<wire x1="68.8" y1="1.8" x2="73.33" y2="1.8" width="0" layer="19" extent="1-16"/>
 <wire x1="73.33" y1="1.8" x2="78.046" y2="1.8" width="0.4" layer="1"/>
 <wire x1="78.046" y1="1.8" x2="78.4" y2="2.154" width="0.3" layer="1"/>
@@
 <wire x1="78.625" y1="4.7" x2="78.9" y2="4.7" width="0.2" layer="1"/>
 <wire x1="78.6" y1="4.675" x2="78.625" y2="4.7" width="0.2" layer="1"/>
-<wire x1="74.7" y1="-4.4" x2="75.6" y2="-5.3" width="0" layer="19" extent="1-16"/>
-<wire x1="68.7262" y1="-4.4" x2="74.7" y2="-4.4" width="0" layer="19" extent="1-16"/>
-<wire x1="68.7012" y1="-4.375" x2="68.7262" y2="-4.4" width="0" layer="19" extent="1-16"/>
 <wire x1="81.4" y1="6.05" x2="81.4" y2="5.1" width="0.5" layer="1"/>
 <wire x1="82.05" y1="6.7" x2="81.4" y2="6.05" width="0.5" layer="1"/>
@@
 <contactref element="C27" pad="2"/>
 <contactref element="IC3" pad="43"/>
+<wire x1="2.8071" y1="22.9216" x2="2.8071" y2="20.9071" width="0.254" layer="16"/>
+<wire x1="2.8071" y1="20.9071" x2="2.5" y2="20.6" width="0.254" layer="16"/>
+<wire x1="2.5" y1="20.6" x2="1" y2="20.6" width="0.254" layer="16"/>
+<via x="1" y="20.6" extent="1-16" drill="0.4"/>
+<wire x1="1" y1="20.6" x2="1" y2="18.8" width="0.254" layer="1"/>
+<wire x1="1" y1="18.8" x2="3.5" y2="16.3" width="0.254" layer="1"/>
+<wire x1="3.5" y1="16.3" x2="5.7" y2="16.3" width="0.254" layer="1"/>
 <wire x1="24.675" y1="5.75" x2="70.5" y2="2.7" width="0" layer="19" extent="1-1"/>
 <wire x1="21.346" y1="2.854" x2="24.675" y2="5.75" width="0" layer="19" extent="1-1"/>
@@
 <wire x1="13.7" y1="5" x2="13.6644" y2="3.2062" width="0" layer="19" extent="1-16"/>
 <wire x1="12.6644" y1="15.2062" x2="22.4144" y2="14.3476" width="0" layer="19" extent="1-1"/>
-<wire x1="12.5" y1="21.6" x2="12.6126" y2="15.258" width="0" layer="19" extent="1-1"/>
-<wire x1="2.8071" y1="22.9216" x2="12.5" y2="21.6" width="0" layer="19" extent="1-16"/>
-<wire x1="-3.519009375" y1="-24.296334375" x2="8" y2="-18.8" width="0" layer="19" extent="1-16"/>
-<wire x1="-3.313796875" y1="-24.86015" x2="-3.519009375" y2="-24.296334375" width="0" layer="19" extent="1-1"/>
+<wire x1="5.7" y1="16.3" x2="11.5432" y2="15.258" width="0" layer="19" extent="1-1"/>
+<wire x1="-3.313796875" y1="-24.86015" x2="-3.519009375" y2="-24.6549375" width="0.254" layer="1"/>
+<wire x1="-3.519009375" y1="-24.6549375" x2="-3.519009375" y2="-24.296334375" width="0.254" layer="1"/>
+<wire x1="-3.519009375" y1="-24.296334375" x2="-1.3" y2="-23.5" width="0.254" layer="1"/>
+<wire x1="-1.3" y1="-23.5" x2="3.4" y2="-18.8" width="0.254" layer="1"/>
+<wire x1="3.4" y1="-18.8" x2="8" y2="-18.8" width="0.254" layer="1"/>
 </signal>
 <signal name="D-">
@@
 <signal name="SS3">
 <contactref element="SD1" pad="2"/>
+<contactref element="IC3" pad="62"/>
+<wire x1="13.6644" y1="15.2062" x2="13.6644" y2="18.6356" width="0.2032" layer="1"/>
+<wire x1="13.6644" y1="18.6356" x2="10.4" y2="21.9" width="0.2032" layer="1"/>
+<via x="10.4" y="21.9" extent="1-16" drill="0.4"/>
+<wire x1="10.4" y1="21.9" x2="8.3" y2="21.9" width="0.2032" layer="16"/>
+<wire x1="8.3" y1="21.9" x2="7.5" y2="21.1" width="0.2032" layer="16"/>
+<wire x1="7.5" y1="21.1" x2="5.2" y2="21.1" width="0.2032" layer="16"/>
+<wire x1="5.2" y1="21.1" x2="5" y2="21.3" width="0.2032" layer="16"/>
+<wire x1="5" y1="21.3" x2="5" y2="22.3145" width="0.2032" layer="16"/>
+<wire x1="5" y1="22.3145" x2="5.0071" y2="22.3216" width="0.2032" layer="16"/>
 </signal>
 <signal name="LED2">
@@
 <contactref element="IC4" pad="2"/>
 <contactref element="R22" pad="1"/>
-<wire x1="62.8" y1="0.3" x2="64.7" y2="0.3" width="0" layer="19" extent="1-16"/>
 <wire x1="64.9" y1="0.5" x2="77.246" y2="0.5" width="0.2" layer="1"/>
-<wire x1="64.7" y1="0.3" x2="64.9" y2="0.5" width="0" layer="19" extent="1-16"/>
-<wire x1="62.8" y1="12.2" x2="62.8" y2="0.3" width="0" layer="19" extent="1-16"/>
 <wire x1="75.7" y1="10.8" x2="77.15" y2="10.8" width="0.2" layer="1"/>
 <wire x1="73.5" y1="13" x2="75.7" y2="10.8" width="0.2" layer="1"/>
 <wire x1="63.6" y1="13" x2="73.5" y2="13" width="0.2" layer="1"/>
 <wire x1="62.8" y1="12.2" x2="63.6" y2="13" width="0.2" layer="1"/>
-<wire x1="62.8" y1="0.3" x2="62.8" y2="0.3" width="0" layer="19" extent="1-16"/>
 <via x="62.8" y="12.2" extent="1-16" drill="0.4" shape="octagon"/>
+<wire x1="77.246" y1="0.5" x2="77.15" y2="10.8" width="0" layer="19" extent="1-1"/>
 </signal>
 <signal name="N$70">
@@
 <wire x1="-18.9435" y1="26.31" x2="-8.6565" y2="26.31" width="0" layer="19" extent="16-16"/>
 </signal>
+<signal name="SW4">
+<contactref element="SW4" pad="1"/>
+<contactref element="IC3" pad="2"/>
+<wire x1="10.4144" y1="12.4562" x2="9.1438" y2="12.4562" width="0.2286" layer="1"/>
+<wire x1="9.1438" y1="12.4562" x2="8.4" y2="13.2" width="0.2286" layer="1"/>
+<wire x1="8.4" y1="13.2" x2="3.7" y2="13.2" width="0.2286" layer="1"/>
+<wire x1="3.7" y1="13.2" x2="0.954" y2="14.388434375" width="0.2286" layer="1"/>
+</signal>
+<signal name="SW3">
+<contactref element="SW3" pad="1"/>
+<contactref element="IC3" pad="59"/>
+<wire x1="3.054" y1="19.888434375" x2="3.054" y2="26.754" width="0.2286" layer="1"/>
+<wire x1="3.054" y1="26.754" x2="3.9" y2="27.6" width="0.2286" layer="1"/>
+<wire x1="3.9" y1="27.6" x2="7.3" y2="27.6" width="0.2286" layer="1"/>
+<wire x1="7.3" y1="27.6" x2="15.1644" y2="19.7356" width="0.2286" layer="1"/>
+<wire x1="15.1644" y1="19.7356" x2="15.1644" y2="15.2062" width="0.2286" layer="1"/>
+</signal>
+<signal name="SW2">
+<contactref element="SW2" pad="1"/>
+<contactref element="IC3" pad="60"/>
+<contactref element="IC3" pad="61"/>
+<wire x1="14.1644" y1="15.2062" x2="14.1644" y2="19.6356" width="0.2286" layer="1"/>
+<wire x1="14.1644" y1="19.6356" x2="10.1" y2="23.7" width="0.2286" layer="1"/>
+<wire x1="10.1" y1="23.7" x2="5.054" y2="25.688434375" width="0.2286" layer="1"/>
+<wire x1="14.6644" y1="15.2062" x2="14.1644" y2="15.2062" width="0.2286" layer="1"/>
+</signal>
 </signals>

Commit message: routing
Connections:
- net CE: now also IC3.49
- net CSN: now also IC3.50
- net IRQ: now also IC3.46
Routing:
- net CE: track 12.8 -> 63.0 mm, vias 0 -> 2
Changed lines of the file:
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@@
 </class>
 </classes>
-<designrules name="default *">
+<designrules>
 <description language="de">&lt;b&gt;EAGLE Design Rules&lt;/b&gt;
 &lt;p&gt;
@@
 <contactref element="IC4" pad="1"/>
 <wire x1="64.4" y1="1" x2="77.246" y2="1" width="0.2" layer="1"/>
+<contactref element="IC3" pad="49"/>
+<wire x1="20.1644" y1="15.2062" x2="21.0938" y2="15.2062" width="0.2286" layer="1"/>
+<wire x1="21.0938" y1="15.2062" x2="21.1" y2="15.2" width="0.2286" layer="1"/>
+<via x="21.1" y="15.2" extent="1-16" drill="0.4"/>
+<wire x1="21.1" y1="15.2" x2="21.7" y2="15.2" width="0.2286" layer="16"/>
+<wire x1="21.7" y1="15.2" x2="26.4" y2="10.5" width="0.2286" layer="16"/>
+<wire x1="26.4" y1="10.5" x2="52.6" y2="10.5" width="0.2286" layer="16"/>
+<wire x1="52.6" y1="10.5" x2="53" y2="10.1" width="0.2286" layer="16"/>
+<via x="53" y="10.1" extent="1-16" drill="0.4"/>
+<wire x1="53" y1="10.1" x2="62.1" y2="1" width="0.2286" layer="1"/>
+<wire x1="62.1" y1="1" x2="64.4" y2="1" width="0.2286" layer="1"/>
 </signal>
 <signal name="CSN">
@@
 <wire x1="62.8" y1="12.2" x2="63.6" y2="13" width="0.2" layer="1"/>
 <via x="62.8" y="12.2" extent="1-16" drill="0.4" shape="octagon"/>
+<contactref element="IC3" pad="50"/>
 <wire x1="77.246" y1="0.5" x2="77.15" y2="10.8" width="0" layer="19" extent="1-1"/>
+<wire x1="19.6644" y1="15.2062" x2="62.8" y2="12.2" width="0" layer="19" extent="1-1"/>
 </signal>
 <signal name="N$70">
@@
 <wire x1="78.3" y1="-1.7" x2="78.4" y2="-1.8" width="0.2" layer="1"/>
 <wire x1="78.4" y1="-1.8" x2="78.4" y2="-2.154" width="0.2" layer="1"/>
+<contactref element="IC3" pad="46"/>
+<wire x1="22.4144" y1="11.9562" x2="65.2" y2="-1.8" width="0" layer="19" extent="1-1"/>
 </signal>
 <signal name="N$10">
