File: eagle/lun1k.brd (EAGLE design)
At the start: 127.6 x 60.4 mm, 94 parts, among them IC1 LTC3558, IC3 STM32F405RGT, IC4 NRF24L01SMD, J2 XF2-3015-1LW, Q1 Q12M-SMD-S, Q2 3.2X2.5CRYSTAL, SW1 JS102011SAQN, SW2 SWITCH_MCTAEF, SW3 SWITCH_MCTAEF, SW4 SWITCH_MCTAEF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

Commit message: routing
Routing:
- net IRQ: track 13.9 -> 68.0 mm, vias 0 -> 2
Changed lines of the file:
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@@
 <signal name="IRQ">
 <contactref element="IC4" pad="6"/>
-<wire x1="65.2" y1="-1.8" x2="65.6" y2="-1.4" width="0.2" layer="1"/>
-<wire x1="65.6" y1="-1.4" x2="75.9" y2="-1.4" width="0.2" layer="1"/>
+<wire x1="65.2" y1="-1.8" x2="65.6" y2="-1.4" width="0" layer="19" extent="1-16"/>
+<wire x1="65.6" y1="-1.4" x2="66.3" y2="-1.4" width="0.2" layer="1"/>
+<wire x1="66.3" y1="-1.4" x2="75.9" y2="-1.4" width="0.2" layer="1"/>
 <wire x1="75.9" y1="-1.4" x2="76.2" y2="-1.7" width="0.2" layer="1"/>
 <wire x1="76.2" y1="-1.7" x2="78.3" y2="-1.7" width="0.2" layer="1"/>
@@
 <wire x1="78.4" y1="-1.8" x2="78.4" y2="-2.154" width="0.2" layer="1"/>
 <contactref element="IC3" pad="46"/>
-<wire x1="22.4144" y1="11.9562" x2="65.2" y2="-1.8" width="0" layer="19" extent="1-1"/>
+<wire x1="22.4144" y1="11.9562" x2="21.3438" y2="11.9562" width="0.2286" layer="1"/>
+<wire x1="21.3438" y1="11.9562" x2="20.8" y2="12.5" width="0.2286" layer="1"/>
+<wire x1="20.8" y1="12.5" x2="20.8" y2="13.6" width="0.2286" layer="1"/>
+<via x="20.8" y="13.6" extent="1-16" drill="0.4"/>
+<wire x1="20.8" y1="13.6" x2="22" y2="13.6" width="0.2286" layer="16"/>
+<wire x1="22" y1="13.6" x2="26" y2="9.6" width="0.2286" layer="16"/>
+<wire x1="26" y1="9.6" x2="47.4" y2="9.6" width="0.2286" layer="16"/>
+<wire x1="47.4" y1="9.6" x2="48.1" y2="8.9" width="0.2286" layer="16"/>
+<via x="48.1" y="8.9" extent="1-16" drill="0.4"/>
+<wire x1="48.1" y1="8.9" x2="58.4" y2="-1.4" width="0.2286" layer="1"/>
+<wire x1="58.4" y1="-1.4" x2="66.3" y2="-1.4" width="0.2286" layer="1"/>
 </signal>
 <signal name="N$10">

Commit message: routing
Routing:
- net CSN: track 27.9 -> 92.2 mm, vias 1 -> 3
Changed lines of the file:
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@@
 <via x="70" y="-10" extent="1-16" drill="0.4" shape="octagon"/>
 <via x="54" y="-10" extent="1-16" drill="0.4" shape="octagon"/>
-<via x="54" y="10" extent="1-16" drill="0.4" shape="octagon"/>
+<via x="57.4" y="10.7" extent="1-16" drill="0.4" shape="octagon"/>
 <via x="42" y="-10" extent="1-16" drill="0.4" shape="octagon"/>
 <via x="42" y="10" extent="1-16" drill="0.4" shape="octagon"/>
@@
 <wire x1="21.1" y1="15.2" x2="21.7" y2="15.2" width="0.2286" layer="16"/>
 <wire x1="21.7" y1="15.2" x2="26.4" y2="10.5" width="0.2286" layer="16"/>
-<wire x1="26.4" y1="10.5" x2="52.6" y2="10.5" width="0.2286" layer="16"/>
-<wire x1="52.6" y1="10.5" x2="53" y2="10.1" width="0.2286" layer="16"/>
-<via x="53" y="10.1" extent="1-16" drill="0.4"/>
-<wire x1="53" y1="10.1" x2="62.1" y2="1" width="0.2286" layer="1"/>
-<wire x1="62.1" y1="1" x2="64.4" y2="1" width="0.2286" layer="1"/>
+<wire x1="26.4" y1="10.5" x2="54.1" y2="10.5" width="0.2286" layer="16"/>
+<wire x1="54.1" y1="10.5" x2="54.5" y2="10.1" width="0.2286" layer="16"/>
+<via x="54.5" y="10.1" extent="1-16" drill="0.4"/>
+<wire x1="54.5" y1="10.1" x2="63.6" y2="1" width="0.2286" layer="1"/>
+<wire x1="63.6" y1="1" x2="64.4" y2="1" width="0.2286" layer="1"/>
 </signal>
 <signal name="CSN">
 <contactref element="IC4" pad="2"/>
 <contactref element="R22" pad="1"/>
-<wire x1="64.9" y1="0.5" x2="77.246" y2="0.5" width="0.2" layer="1"/>
 <wire x1="75.7" y1="10.8" x2="77.15" y2="10.8" width="0.2" layer="1"/>
 <wire x1="73.5" y1="13" x2="75.7" y2="10.8" width="0.2" layer="1"/>
@@
 <via x="62.8" y="12.2" extent="1-16" drill="0.4" shape="octagon"/>
 <contactref element="IC3" pad="50"/>
-<wire x1="77.246" y1="0.5" x2="77.15" y2="10.8" width="0" layer="19" extent="1-1"/>
-<wire x1="19.6644" y1="15.2062" x2="62.8" y2="12.2" width="0" layer="19" extent="1-1"/>
+<wire x1="19.6644" y1="15.2062" x2="19.6644" y2="13.5644" width="0.2286" layer="1"/>
+<wire x1="19.6644" y1="13.5644" x2="19.4" y2="13.3" width="0.2286" layer="1"/>
+<via x="19.4" y="13.3" extent="1-16" drill="0.4"/>
+<wire x1="19.4" y1="13.3" x2="20.2" y2="12.5" width="0.2286" layer="16"/>
+<wire x1="20.2" y1="12.5" x2="22.1" y2="12.5" width="0.2286" layer="16"/>
+<wire x1="22.1" y1="12.5" x2="25.9" y2="8.7" width="0.2286" layer="16"/>
+<wire x1="25.9" y1="8.7" x2="52.8" y2="8.7" width="0.2286" layer="16"/>
+<wire x1="52.8" y1="8.7" x2="54.2" y2="8.7" width="0.2286" layer="16"/>
+<wire x1="54.2" y1="8.7" x2="59.3" y2="8.7" width="0.2286" layer="16"/>
+<wire x1="59.3" y1="8.7" x2="62.8" y2="12.2" width="0.2286" layer="16"/>
+<wire x1="77.246" y1="0.5" x2="62.5" y2="0.5" width="0.2286" layer="1"/>
+<wire x1="62.5" y1="0.5" x2="61.2" y2="1.8" width="0.2286" layer="1"/>
+<wire x1="61.2" y1="1.8" x2="54.3" y2="8.7" width="0.2286" layer="1"/>
+<wire x1="54.3" y1="8.7" x2="54.2" y2="8.7" width="0.2286" layer="1"/>
+<via x="54.2" y="8.7" extent="1-16" drill="0.4"/>
+<wire x1="54.2" y1="8.7" x2="52.8" y2="8.7" width="0.2286" layer="16"/>
 </signal>
 <signal name="N$70">

Commit message: routing
Routing:
- net +3V3: track 76.5 -> 145.6 mm, vias 2 -> 3
Changed lines of the file:
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@@
 <via x="80.22" y="-0.875" extent="1-16" drill="0.4" shape="octagon" alwaysstop="yes"/>
 <via x="68.7012" y="-4.375" extent="1-16" drill="0.4" shape="octagon"/>
-<via x="68.8" y="1.8" extent="1-16" drill="0.4" shape="octagon"/>
+<via x="66.9" y="3.3" extent="1-16" drill="0.4" shape="octagon"/>
 <via x="78.58" y="0.875" extent="1-16" drill="0.4" shape="octagon" alwaysstop="yes"/>
 <via x="80.22" y="0.875" extent="1-16" drill="0.4" shape="octagon" alwaysstop="yes"/>
@@
 <via x="57.4" y="10.7" extent="1-16" drill="0.4" shape="octagon"/>
 <via x="42" y="-10" extent="1-16" drill="0.4" shape="octagon"/>
-<via x="42" y="10" extent="1-16" drill="0.4" shape="octagon"/>
-<via x="46.2" y="8" extent="1-16" drill="0.4" shape="octagon"/>
+<via x="43.8" y="5.4" extent="1-16" drill="0.4" shape="octagon"/>
+<via x="46.3" y="5.7" extent="1-16" drill="0.4" shape="octagon"/>
 <via x="48" y="-10" extent="1-16" drill="0.4" shape="octagon"/>
 <via x="60" y="-10" extent="1-16" drill="0.4" shape="octagon"/>
-<via x="60" y="6" extent="1-16" drill="0.4" shape="octagon"/>
+<via x="63.2" y="5.7" extent="1-16" drill="0.4" shape="octagon"/>
 <via x="66" y="10" extent="1-16" drill="0.4" shape="octagon"/>
 <via x="66" y="-10" extent="1-16" drill="0.4" shape="octagon"/>
-<via x="60" y="10" extent="1-16" drill="0.4" shape="octagon"/>
+<via x="63.7" y="9.6" extent="1-16" drill="0.4" shape="octagon"/>
 <via x="88.55" y="-6.4" extent="1-16" drill="0.4" shape="octagon"/>
 <via x="88.55" y="-8.4" extent="1-16" drill="0.4" shape="octagon"/>
@@
 <signal name="+3V3" class="2">
 <contactref element="FERRITE" pad="1"/>
-<wire x1="70.5" y1="2.7" x2="75.4" y2="7.6" width="0.3" layer="1"/>
 <wire x1="75.4" y1="7.6" x2="77.2" y2="7.6" width="0.3" layer="1"/>
 <wire x1="77.2" y1="7.6" x2="77.3" y2="7.7" width="0.3" layer="1"/>
@@
 <wire x1="8" y1="-17.5" x2="8" y2="-18.8" width="0.3048" layer="1"/>
 <via x="8" y="-18.8" extent="1-16" drill="0.6"/>
-<wire x1="8" y1="-18.8" x2="8" y2="-0.7" width="0.3048" layer="16"/>
+<wire x1="8" y1="-18.8" x2="8" y2="-6" width="0.3048" layer="16"/>
+<wire x1="8" y1="-6" x2="8" y2="-0.7" width="0.3048" layer="16"/>
 <wire x1="8" y1="-0.7" x2="13.7" y2="5" width="0.3048" layer="16"/>
 <contactref element="J2" pad="13"/>
@@
 <wire x1="1" y1="18.8" x2="3.5" y2="16.3" width="0.254" layer="1"/>
 <wire x1="3.5" y1="16.3" x2="5.7" y2="16.3" width="0.254" layer="1"/>
-<wire x1="24.675" y1="5.75" x2="70.5" y2="2.7" width="0" layer="19" extent="1-1"/>
-<wire x1="21.346" y1="2.854" x2="24.675" y2="5.75" width="0" layer="19" extent="1-1"/>
-<wire x1="24.675" y1="-0.75" x2="21.346" y2="2.1804" width="0" layer="19" extent="1-1"/>
-<wire x1="24.675" y1="-1.25" x2="24.675" y2="-0.75" width="0" layer="19" extent="1-1"/>
-<wire x1="24.675" y1="-5.75" x2="24.675" y2="-1.25" width="0" layer="19" extent="1-1"/>
-<wire x1="22.4144" y1="10.4562" x2="24.675" y2="5.75" width="0" layer="19" extent="1-1"/>
-<wire x1="22.4144" y1="12.9562" x2="22.4144" y2="10.4562" width="0" layer="19" extent="1-1"/>
-<wire x1="13.6644" y1="3.2062" x2="20.1644" y2="3.2062" width="0" layer="19" extent="1-1"/>
-<wire x1="13.7" y1="5" x2="13.6644" y2="3.2062" width="0" layer="19" extent="1-16"/>
-<wire x1="12.6644" y1="15.2062" x2="22.4144" y2="14.3476" width="0" layer="19" extent="1-1"/>
-<wire x1="5.7" y1="16.3" x2="11.5432" y2="15.258" width="0" layer="19" extent="1-1"/>
 <wire x1="-3.313796875" y1="-24.86015" x2="-3.519009375" y2="-24.6549375" width="0.254" layer="1"/>
 <wire x1="-3.519009375" y1="-24.6549375" x2="-3.519009375" y2="-24.296334375" width="0.254" layer="1"/>
@@
 <wire x1="-1.3" y1="-23.5" x2="3.4" y2="-18.8" width="0.254" layer="1"/>
 <wire x1="3.4" y1="-18.8" x2="8" y2="-18.8" width="0.254" layer="1"/>
+<wire x1="75.4" y1="7.6" x2="66.3" y2="7.6" width="0.3048" layer="1"/>
+<wire x1="66.3" y1="7.6" x2="59.3" y2="7.6" width="0.3048" layer="1"/>
+<wire x1="59.3" y1="7.6" x2="59.2" y2="7.5" width="0.3048" layer="1"/>
+<via x="59.2" y="7.5" extent="1-16" drill="0.4"/>
+<wire x1="59.2" y1="7.5" x2="31.5" y2="7.5" width="0.3048" layer="16"/>
+<wire x1="31.5" y1="7.5" x2="29.7" y2="5.7" width="0.3048" layer="16"/>
+<wire x1="29.7" y1="5.7" x2="29.7" y2="0.7" width="0.3048" layer="16"/>
+<wire x1="29.7" y1="0.7" x2="25.1" y2="-3.9" width="0.3048" layer="16"/>
+<wire x1="25.1" y1="-3.9" x2="24" y2="-3.9" width="0.3048" layer="16"/>
+<wire x1="24" y1="-3.9" x2="21.7" y2="-6.2" width="0.3048" layer="16"/>
+<wire x1="21.7" y1="-6.2" x2="8.2" y2="-6.2" width="0.3048" layer="16"/>
+<wire x1="8.2" y1="-6.2" x2="8" y2="-6" width="0.3048" layer="16"/>
+<wire x1="22.4144" y1="10.4562" x2="22.4144" y2="12.9562" width="0" layer="19" extent="1-1"/>
+<wire x1="24.675" y1="5.75" x2="22.4144" y2="10.4562" width="0" layer="19" extent="1-1"/>
+<wire x1="21.346" y1="2.854" x2="24.675" y2="5.75" width="0" layer="19" extent="1-1"/>
+<wire x1="24.675" y1="-0.75" x2="21.346" y2="2.1804" width="0" layer="19" extent="1-1"/>
+<wire x1="24.675" y1="-1.25" x2="24.675" y2="-0.75" width="0" layer="19" extent="1-1"/>
+<wire x1="25.1" y1="-3.9" x2="24.675" y2="-1.25" width="0" layer="19" extent="1-16"/>
+<wire x1="13.6644" y1="3.2062" x2="13.7" y2="5" width="0" layer="19" extent="1-16"/>
+<wire x1="24.675" y1="-5.75" x2="25.1" y2="-3.9" width="0" layer="19" extent="1-16"/>
+<wire x1="12.6644" y1="15.2062" x2="22.4144" y2="14.3476" width="0" layer="19" extent="1-1"/>
+<wire x1="5.7" y1="16.3" x2="11.5432" y2="15.258" width="0" layer="19" extent="1-1"/>
 </signal>
 <signal name="D-">
