File: eagle/lun1k.brd (EAGLE design)
At the start: 127.6 x 60.4 mm, 94 parts, among them IC1 LTC3558, IC3 STM32F405RGT, IC4 NRF24L01SMD, J2 XF2-3015-1LW, Q1 Q12M-SMD-S, Q2 3.2X2.5CRYSTAL, SW1 JS102011SAQN, SW2 SWITCH_MCTAEF, SW3 SWITCH_MCTAEF, SW4 SWITCH_MCTAEF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

Commit message: routing
Parts:
- moved C30 49.5 mm to (19.0, -5.72), turned to 180 degrees
- moved C29 22.1 mm to (49.0, 18.6), turned to 0 degrees
- moved C28 14.1 mm to (43.0, 18.6), turned to 180 degrees
Routing:
- net +3V3: track 145.6 -> 197.6 mm, vias 3 -> 7
- net VCOMH: track 0.00 -> 33.6 mm, vias 0 -> 2
- net +12V: track 26.3 -> 52.1 mm, vias 2 -> 3
- net GND: track 58.5 -> 55.8 mm
- net IRQ: track 68.0 -> 66.8 mm
- net CSN: track 92.2 -> 93.2 mm

Commit message: routing
Connections:
- removed net D8: J2.25
- net GND: now also J2.25
Routing:
- net +3V3: track 197.6 -> 209.2 mm, vias 7 -> 10
- net GND: track 55.8 -> 62.7 mm
Changed lines of the file:
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@@
 <contactref element="IC3" pad="1"/>
 </signal>
-<signal name="GND" class="2" airwireshidden="yes">
+<signal name="GND" class="2">
 <contactref element="X1" pad="GND"/>
 <contactref element="LED1" pad="C"/>
@@
 <contactref element="X1_" pad="2"/>
 <contactref element="C27" pad="1"/>
-<wire x1="36.3" y1="16" x2="36.4" y2="16.1" width="0" layer="19" extent="1-16"/>
 <wire x1="77.2217" y1="4.675" x2="78.6" y2="4.675" width="0.2" layer="1"/>
 <wire x1="78.3892" y1="2.154" x2="78.354" y2="2.154" width="0.2" layer="1"/>
@@
 <wire x1="76.205" y1="4.675" x2="77.2217" y2="4.675" width="0.4" layer="1"/>
 <wire x1="73.33" y1="1.8" x2="76.205" y2="4.675" width="0.4" layer="1"/>
-<wire x1="36.4" y1="16.1" x2="36.2" y2="16.3" width="0" layer="19" extent="1-16"/>
-<wire x1="36.2" y1="16.3" x2="35" y2="16.3" width="0" layer="19" extent="1-16"/>
-<wire x1="35" y1="16.3" x2="34.6526" y2="16.6474" width="0" layer="19" extent="1-16"/>
-<wire x1="34.6526" y1="16.6474" x2="34.65269375" y2="17.283434375" width="0" layer="19" extent="1-16"/>
 <wire x1="77.4" y1="-4.2" x2="77.3" y2="-4.3" width="0.2" layer="1"/>
 <wire x1="77.2217" y1="4.675" x2="77.2217" y2="4.4217" width="0.2" layer="1"/>
@@
 <via x="16.3" y="-15" extent="1-16" drill="0.6"/>
 <contactref element="U1" pad="9"/>
+<wire x1="24.675" y1="-6.25" x2="25.85" y2="-6.25" width="0.254" layer="1"/>
+<wire x1="24.775" y1="-7.25" x2="25.95" y2="-7.25" width="0.254" layer="1"/>
+<wire x1="24.675" y1="-1.75" x2="23.45" y2="-1.75" width="0.254" layer="1"/>
+<wire x1="23.45" y1="-1.75" x2="23.45" y2="-1.65" width="0.254" layer="1"/>
+<wire x1="23.45" y1="-1.65" x2="23.3" y2="-1.5" width="0.254" layer="1"/>
+<contactref element="J2" pad="25"/>
+<wire x1="24.675" y1="4.75" x2="26.75" y2="4.75" width="0.254" layer="1"/>
+<wire x1="26.75" y1="4.75" x2="27.4" y2="4.1" width="0.254" layer="1"/>
 <wire x1="13.1644" y1="15.2062" x2="16.1644" y2="15.2062" width="0" layer="19" extent="1-1"/>
 <wire x1="10.2432" y1="15.258" x2="13.1644" y2="15.2062" width="0" layer="19" extent="1-1"/>
-<wire x1="24.675" y1="-6.25" x2="24.675" y2="-7.25" width="0" layer="19" extent="1-1"/>
 <wire x1="13.1644" y1="3.2062" x2="13.6646" y2="0.2898" width="0" layer="19" extent="1-1"/>
 <wire x1="18.1644" y1="3.2062" x2="21.346" y2="0.8804" width="0" layer="19" extent="1-1"/>
-<wire x1="24.675" y1="-1.75" x2="21.346" y2="0.8804" width="0" layer="19" extent="1-1"/>
 </signal>
 <signal name="+5V" class="1">
@@
 <via x="59.9" y="6.7" extent="1-16" drill="0.4"/>
 <wire x1="59.9" y1="6.7" x2="30.7" y2="6.7" width="0.3048" layer="16"/>
-<wire x1="30.7" y1="6.7" x2="29.7" y2="5.7" width="0.3048" layer="16"/>
+<wire x1="30.7" y1="6.7" x2="30.5" y2="6.5" width="0.3048" layer="16"/>
+<wire x1="30.5" y1="6.5" x2="30.2" y2="6.2" width="0.3048" layer="16"/>
+<wire x1="30.2" y1="6.2" x2="29.7" y2="5.7" width="0.3048" layer="16"/>
 <wire x1="29.7" y1="5.7" x2="29.7" y2="0.7" width="0.3048" layer="16"/>
-<wire x1="29.7" y1="0.7" x2="25.1" y2="-3.9" width="0.3048" layer="16"/>
+<wire x1="29.7" y1="0.7" x2="26.9" y2="-2.1" width="0.3048" layer="16"/>
+<wire x1="26.9" y1="-2.1" x2="26.85" y2="-2.15" width="0.3048" layer="16"/>
+<wire x1="26.85" y1="-2.15" x2="25.1" y2="-3.9" width="0.3048" layer="16"/>
 <wire x1="25.1" y1="-3.9" x2="24" y2="-3.9" width="0.3048" layer="16"/>
-<wire x1="24" y1="-3.9" x2="21.7" y2="-6.2" width="0.3048" layer="16"/>
+<wire x1="24" y1="-3.9" x2="22.9" y2="-5" width="0.3048" layer="16"/>
+<wire x1="22.9" y1="-5" x2="22.75" y2="-5.15" width="0.3048" layer="16"/>
+<wire x1="22.75" y1="-5.15" x2="21.7" y2="-6.2" width="0.3048" layer="16"/>
 <wire x1="21.7" y1="-6.2" x2="8.2" y2="-6.2" width="0.3048" layer="16"/>
 <wire x1="8.2" y1="-6.2" x2="8" y2="-6" width="0.3048" layer="16"/>
@@
 <wire x1="20.5" y1="13.8" x2="20.8" y2="13.8" width="0.2286" layer="1"/>
 <wire x1="20.8" y1="13.8" x2="21.1" y2="14.1" width="0.2286" layer="1"/>
-<wire x1="20.4" y1="5.5" x2="24.675" y2="5.75" width="0" layer="19" extent="1-1"/>
-<wire x1="24.675" y1="-5.75" x2="25.1" y2="-3.9" width="0" layer="19" extent="1-16"/>
-<wire x1="24.675" y1="-1.25" x2="25.1" y2="-3.9" width="0" layer="19" extent="1-16"/>
-<wire x1="24.675" y1="-0.75" x2="24.675" y2="-1.25" width="0" layer="19" extent="1-1"/>
+<wire x1="24.675" y1="-5.75" x2="23.65" y2="-5.75" width="0.254" layer="1"/>
+<wire x1="23.65" y1="-5.75" x2="22.9" y2="-5" width="0.254" layer="1"/>
+<via x="22.9" y="-5" extent="1-16" drill="0.4"/>
+<wire x1="22.9" y1="-5" x2="22.75" y2="-5.15" width="0.254" layer="16"/>
+<wire x1="24.675" y1="-0.75" x2="24.675" y2="-1.25" width="0.254" layer="1"/>
+<wire x1="24.675" y1="-1.25" x2="25.95" y2="-1.25" width="0.254" layer="1"/>
+<wire x1="25.95" y1="-1.25" x2="26.5" y2="-1.8" width="0.254" layer="1"/>
+<via x="26.5" y="-1.8" extent="1-16" drill="0.4"/>
+<wire x1="26.5" y1="-1.8" x2="26.9" y2="-2.1" width="0.254" layer="16"/>
+<wire x1="26.9" y1="-2.1" x2="26.85" y2="-2.15" width="0.254" layer="16"/>
+<wire x1="24.675" y1="5.75" x2="29.75" y2="5.75" width="0.254" layer="1"/>
+<wire x1="29.75" y1="5.75" x2="30.2" y2="6.2" width="0.254" layer="1"/>
+<via x="30.2" y="6.2" extent="1-16" drill="0.4"/>
+<wire x1="30.2" y1="6.2" x2="30.5" y2="6.5" width="0.254" layer="16"/>
 </signal>
 <signal name="D-">
@@
 <contactref element="J2" pad="11"/>
 <contactref element="IC3" pad="25"/>
-<wire x1="24.675" y1="-2.25" x2="22.15" y2="-2.25" width="0.254" layer="1"/>
-<wire x1="22.15" y1="-2.25" x2="22" y2="-2.2" width="0.254" layer="1"/>
-<via x="22" y="-2.2" extent="1-16" drill="0.4"/>
-<wire x1="22" y1="-2.2" x2="21.4" y2="-2.8" width="0.254" layer="16"/>
-<wire x1="21.4" y1="-2.8" x2="18.4" y2="-2.8" width="0.254" layer="16"/>
+<wire x1="24.675" y1="-2.25" x2="21.45" y2="-2.25" width="0.254" layer="1"/>
+<wire x1="21.45" y1="-2.25" x2="21.2" y2="-2.5" width="0.254" layer="1"/>
+<via x="21.2" y="-2.5" extent="1-16" drill="0.4"/>
+<wire x1="21.2" y1="-2.5" x2="20.9" y2="-2.8" width="0.254" layer="16"/>
+<wire x1="20.9" y1="-2.8" x2="18.4" y2="-2.8" width="0.254" layer="16"/>
 <wire x1="18.4" y1="-2.8" x2="16.2" y2="-0.6" width="0.254" layer="16"/>
 <wire x1="16.2" y1="-0.6" x2="16.2" y2="4.8" width="0.254" layer="16"/>
@@
 <wire x1="22.4144" y1="4.7856" x2="22.4144" y2="5.4562" width="0.2032" layer="1"/>
 </signal>
-<signal name="D8">
-<contactref element="J2" pad="25"/>
-</signal>
 <signal name="R/W" class="2">
 <contactref element="J2" pad="15"/>
 <contactref element="IC3" pad="40"/>
-<wire x1="24.675" y1="-0.25" x2="25.95" y2="-0.25" width="0.2032" layer="1"/>
-<wire x1="25.95" y1="-0.25" x2="26.6" y2="-0.9" width="0.2032" layer="1"/>
-<via x="26.6" y="-0.9" extent="1-16" drill="0.4"/>
-<wire x1="26.6" y1="-0.9" x2="28.1" y2="0.6" width="0.2032" layer="16"/>
-<wire x1="28.1" y1="0.6" x2="28.1" y2="4.3" width="0.2032" layer="16"/>
+<wire x1="24.675" y1="-0.25" x2="26.25" y2="-0.25" width="0.2032" layer="1"/>
+<wire x1="26.25" y1="-0.25" x2="26.7" y2="-0.7" width="0.2032" layer="1"/>
+<via x="26.7" y="-0.7" extent="1-16" drill="0.4"/>
+<wire x1="26.7" y1="-0.7" x2="28.1" y2="0.7" width="0.2032" layer="16"/>
+<wire x1="28.1" y1="0.7" x2="28.1" y2="4.3" width="0.2032" layer="16"/>
 <wire x1="28.1" y1="4.3" x2="27.1" y2="5.3" width="0.2032" layer="16"/>
 <wire x1="27.1" y1="5.3" x2="25.3" y2="5.3" width="0.2032" layer="16"/>

Commit message: routing
Parts:
- moved C39 0.30 mm to (14.0, 0.94)
- moved C38 0.10 mm to (21.4, 1.53)
- moved C40 0.10 mm to (19.9, 0.33)
Routing:
- net GND: track 62.7 -> 78.3 mm, vias 66 -> 114

Commit message: routing
Routing:
- net +5V: track 38.9 -> 66.8 mm, vias 2 -> 4
- net R/W: track 21.9 -> 24.7 mm
- net +3V3: track 209.6 -> 211.0 mm
- net GND: track 78.3 -> 77.6 mm, vias 114 -> 119
Changed lines of the file:
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@@
 <wire x1="18.6" y1="4.6" x2="18.6" y2="5.7" width="0.254" layer="1"/>
 <wire x1="18.6" y1="5.7" x2="17.9" y2="6.4" width="0.254" layer="1"/>
-<via x="17.9" y="6.4" extent="1-16" drill="0.4"/>
-<wire x1="17.9" y1="6.4" x2="17.2" y2="6.4" width="0.254" layer="16"/>
 <wire x1="18.1644" y1="4.1644" x2="18.1644" y2="3.2062" width="0.254" layer="1"/>
 <wire x1="18.1644" y1="3.2062" x2="18.1644" y2="2.7" width="0.254" layer="1"/>
@@
 <via x="12.4" y="-11.4" extent="1-16" drill="0.4"/>
 <via x="12" y="-8.6" extent="1-16" drill="0.4"/>
-<via x="15.1" y="-7.7" extent="1-16" drill="0.4"/>
+<via x="14.2" y="-7.2" extent="1-16" drill="0.4"/>
 <via x="18.5" y="-7.7" extent="1-16" drill="0.4"/>
 <via x="20.4" y="-9.7" extent="1-16" drill="0.4"/>
@@
 <via x="23.5" y="-20.5" extent="1-16" drill="0.4"/>
 <via x="29.9" y="-20.5" extent="1-16" drill="0.4"/>
-<via x="15.6" y="-5" extent="1-16" drill="0.4"/>
+<via x="15.2" y="-3.9" extent="1-16" drill="0.4"/>
 <via x="12.2" y="1.5" extent="1-16" drill="0.4"/>
 <via x="9.1" y="-4.8" extent="1-16" drill="0.4"/>
@@
 <via x="40.3" y="-23.4" extent="1-16" drill="0.4"/>
 <via x="38.9" y="-14.6" extent="1-16" drill="0.4"/>
+<via x="13" y="-1.1" extent="1-16" drill="0.4"/>
+<via x="16.4" y="7" extent="1-16" drill="0.4"/>
 <wire x1="13.1644" y1="3.2062" x2="13.1644" y2="3.3644" width="0" layer="19" extent="1-1"/>
+<via x="16.9" y="9" extent="1-16" drill="0.4"/>
+<via x="13.3" y="6.8" extent="1-16" drill="0.4"/>
+<via x="18.8" y="11.8" extent="1-16" drill="0.4"/>
+<via x="13.9" y="13.6" extent="1-16" drill="0.4"/>
 </signal>
 <signal name="+5V" class="1">
@@
 <wire x1="18.1" y1="-12.7" x2="18.1" y2="-11.6" width="0.2032" layer="1"/>
 <wire x1="17.8" y1="-9.6" x2="17.6" y2="-9.4" width="0.2032" layer="1"/>
-<wire x1="17.6" y1="-9.4" x2="13.7" y2="-9.4" width="0.2032" layer="1"/>
+<wire x1="17.6" y1="-9.4" x2="15.2" y2="-9.4" width="0.2032" layer="1"/>
+<wire x1="15.2" y1="-9.4" x2="13.7" y2="-9.4" width="0.2032" layer="1"/>
 <wire x1="15.5" y1="-13.6" x2="15.4" y2="-13.6" width="0.2032" layer="1"/>
 <wire x1="15.4" y1="-13.6" x2="15.4" y2="-12.9" width="0.3048" layer="1"/>
@@
 <wire x1="32.5" y1="-13" x2="34" y2="-13" width="0.4064" layer="1"/>
 <contactref element="IC3" pad="42"/>
-<wire x1="17.6" y1="-9.4" x2="22.4144" y2="9.9562" width="0" layer="19" extent="1-1"/>
+<wire x1="22.4144" y1="9.9562" x2="20.3438" y2="9.9562" width="0.2286" layer="1"/>
+<wire x1="20.3438" y1="9.9562" x2="19.6" y2="10.7" width="0.2286" layer="1"/>
+<via x="19.6" y="10.7" extent="1-16" drill="0.4"/>
+<wire x1="19.6" y1="10.7" x2="19" y2="10.7" width="0.2286" layer="16"/>
+<wire x1="19" y1="10.7" x2="17.9" y2="9.6" width="0.2286" layer="16"/>
+<wire x1="17.9" y1="9.6" x2="17.9" y2="7.7" width="0.2286" layer="16"/>
+<wire x1="17.9" y1="7.7" x2="17.9" y2="7.1" width="0.2286" layer="16"/>
+<wire x1="17.9" y1="7.1" x2="16.9" y2="6.1" width="0.2286" layer="16"/>
+<wire x1="16.9" y1="6.1" x2="16.3" y2="6.1" width="0.2286" layer="16"/>
+<wire x1="16.3" y1="6.1" x2="15.5" y2="5.3" width="0.2286" layer="16"/>
+<wire x1="15.5" y1="5.3" x2="15.5" y2="3.2" width="0.2286" layer="16"/>
+<wire x1="15.5" y1="3.2" x2="14.2" y2="1.9" width="0.2286" layer="16"/>
+<wire x1="14.2" y1="1.9" x2="14.2" y2="-0.9" width="0.2286" layer="16"/>
+<wire x1="14.2" y1="-0.9" x2="16.7" y2="-3.4" width="0.2286" layer="16"/>
+<wire x1="16.7" y1="-3.4" x2="16.7" y2="-4.3" width="0.2286" layer="16"/>
+<wire x1="16.7" y1="-4.3" x2="15.6" y2="-5.4" width="0.2286" layer="16"/>
+<via x="15.6" y="-5.4" extent="1-16" drill="0.4"/>
+<wire x1="15.6" y1="-5.4" x2="15.6" y2="-6.3" width="0.2286" layer="1"/>
+<wire x1="15.6" y1="-6.3" x2="15.2" y2="-6.7" width="0.2286" layer="1"/>
+<wire x1="15.2" y1="-6.7" x2="15.2" y2="-9.4" width="0.2286" layer="1"/>
 </signal>
 <signal name="+3V3" class="2">
@@
 <wire x1="13.6644" y1="3.2062" x2="13.6644" y2="5" width="0.2286" layer="1"/>
 <wire x1="13.6644" y1="5" x2="13.6644" y2="5.5644" width="0.2286" layer="1"/>
-<wire x1="13.6644" y1="5.5644" x2="14.3" y2="6.2" width="0.2286" layer="1"/>
-<wire x1="14.3" y1="6.2" x2="19.7" y2="6.2" width="0.2286" layer="1"/>
-<wire x1="19.7" y1="6.2" x2="20.4" y2="5.5" width="0.2286" layer="1"/>
+<wire x1="13.6644" y1="5.5644" x2="16" y2="7.9" width="0.2286" layer="1"/>
+<wire x1="16" y1="7.9" x2="18" y2="7.9" width="0.2286" layer="1"/>
+<wire x1="18" y1="7.9" x2="20.4" y2="5.5" width="0.2286" layer="1"/>
 <wire x1="20.4" y1="5.5" x2="20.4" y2="4.6" width="0.2286" layer="1"/>
 <wire x1="20.4" y1="4.6" x2="20.3" y2="4.5" width="0.2286" layer="1"/>
@@
 <wire x1="18.9" y1="0.1" x2="17.6" y2="1.4" width="0.2032" layer="16"/>
 <wire x1="17.6" y1="1.4" x2="17.6" y2="4.7" width="0.2032" layer="16"/>
-<wire x1="17.6" y1="4.7" x2="18" y2="5.1" width="0.2032" layer="16"/>
-<via x="18" y="5.1" extent="1-16" drill="0.4"/>
-<wire x1="18" y1="5.1" x2="17.6644" y2="4.7644" width="0.2032" layer="1"/>
-<wire x1="17.6644" y1="4.7644" x2="17.6644" y2="3.2062" width="0.2032" layer="1"/>
+<wire x1="17.6" y1="4.7" x2="17.6" y2="5.2" width="0.2032" layer="16"/>
+<via x="17.6" y="5.2" extent="1-16" drill="0.4"/>
+<wire x1="17.6" y1="5.2" x2="17.6644" y2="5.0644" width="0.2032" layer="1"/>
+<wire x1="17.6644" y1="5.0644" x2="17.6644" y2="3.2062" width="0.2032" layer="1"/>
 </signal>
 <signal name="VSL">
@@
 <wire x1="22.8" y1="2.9" x2="22.8" y2="3.3" width="0.254" layer="16"/>
 <wire x1="22.8" y1="3.3" x2="19.4" y2="6.7" width="0.254" layer="16"/>
-<wire x1="19.4" y1="6.7" x2="19.4" y2="7.4" width="0.254" layer="16"/>
-<wire x1="19.4" y1="7.4" x2="20.3" y2="8.3" width="0.254" layer="16"/>
-<via x="20.3" y="8.3" extent="1-16" drill="0.4"/>
+<wire x1="19.4" y1="6.7" x2="19.4" y2="7.5" width="0.254" layer="16"/>
+<wire x1="19.4" y1="7.5" x2="20" y2="8.1" width="0.254" layer="16"/>
+<wire x1="20" y1="8.1" x2="20.5" y2="8.1" width="0.254" layer="16"/>
+<via x="20.5" y="8.1" extent="1-16" drill="0.4"/>
 <contactref element="IC3" pad="36"/>
 <wire x1="22.4144" y1="6.9562" x2="21.6438" y2="6.9562" width="0.2032" layer="1"/>
-<wire x1="21.6438" y1="6.9562" x2="20.3" y2="8.3" width="0.2032" layer="1"/>
+<wire x1="21.6438" y1="6.9562" x2="20.5" y2="8.1" width="0.2032" layer="1"/>
 </signal>
 <signal name="D5">
@@
 <wire x1="24.9" y1="8.1" x2="24.9" y2="8.8" width="0.2032" layer="16"/>
 <wire x1="24.9" y1="8.8" x2="24.3" y2="9.4" width="0.2032" layer="16"/>
-<wire x1="24.3" y1="9.4" x2="20.8" y2="9.4" width="0.2032" layer="16"/>
-<wire x1="20.8" y1="9.4" x2="20.6" y2="9.6" width="0.2032" layer="16"/>
-<via x="20.6" y="9.6" extent="1-16" drill="0.4"/>
-<wire x1="20.6" y1="9.6" x2="21.2438" y2="8.9562" width="0.2032" layer="1"/>
-<wire x1="21.2438" y1="8.9562" x2="22.4144" y2="8.9562" width="0.2032" layer="1"/>
+<wire x1="24.3" y1="9.4" x2="19.4" y2="9.4" width="0.2032" layer="16"/>
+<wire x1="19.4" y1="9.4" x2="19.2" y2="9.6" width="0.2032" layer="16"/>
+<via x="19.2" y="9.6" extent="1-16" drill="0.4"/>
+<wire x1="19.2" y1="9.6" x2="19.8438" y2="8.9562" width="0.2032" layer="1"/>
+<wire x1="19.8438" y1="8.9562" x2="22.4144" y2="8.9562" width="0.2032" layer="1"/>
 </signal>
 <signal name="E" class="2">

Commit message: routing
Routing:
- net GND: track 77.6 -> 79.7 mm
- net VLIPO: track 62.6 -> 63.9 mm
- net +12V: track 52.1 -> 53.1 mm
- net CSN: track 93.2 -> 92.6 mm
Changed lines of the file:
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@@
 <layer number="14" name="Route14" color="1" fill="6" visible="no" active="no"/>
 <layer number="15" name="Route15" color="4" fill="6" visible="no" active="no"/>
-<layer number="16" name="Bottom" color="1" fill="1" visible="yes" active="yes"/>
+<layer number="16" name="Bottom" color="1" fill="1" visible="no" active="yes"/>
 <layer number="17" name="Pads" color="2" fill="1" visible="yes" active="yes"/>
 <layer number="18" name="Vias" color="2" fill="1" visible="yes" active="yes"/>
@@
 <wire x1="24.675" y1="-6.25" x2="25.85" y2="-6.25" width="0.254" layer="1"/>
 <wire x1="24.775" y1="-7.25" x2="25.95" y2="-7.25" width="0.254" layer="1"/>
-<wire x1="24.675" y1="-1.75" x2="23.45" y2="-1.75" width="0.254" layer="1"/>
+<wire x1="24.675" y1="-1.75" x2="24.35" y2="-1.75" width="0.254" layer="1"/>
+<wire x1="24.35" y1="-1.75" x2="23.45" y2="-1.75" width="0.254" layer="1"/>
 <wire x1="23.45" y1="-1.75" x2="23.45" y2="-1.65" width="0.254" layer="1"/>
 <wire x1="23.45" y1="-1.65" x2="23.3" y2="-1.5" width="0.254" layer="1"/>
@@
 <via x="27.2" y="-12.9" extent="1-16" drill="0.4"/>
 <via x="28.9" y="-15.2" extent="1-16" drill="0.4"/>
-<via x="24.5" y="-16" extent="1-16" drill="0.4"/>
+<via x="18.1" y="-23.5" extent="1-16" drill="0.4"/>
 <via x="31.1" y="-16.8" extent="1-16" drill="0.4"/>
 <via x="23.5" y="-20.5" extent="1-16" drill="0.4"/>
@@
 <via x="13" y="-1.1" extent="1-16" drill="0.4"/>
 <via x="16.4" y="7" extent="1-16" drill="0.4"/>
-<wire x1="13.1644" y1="3.2062" x2="13.1644" y2="3.3644" width="0" layer="19" extent="1-1"/>
 <via x="16.9" y="9" extent="1-16" drill="0.4"/>
 <via x="13.3" y="6.8" extent="1-16" drill="0.4"/>
 <via x="18.8" y="11.8" extent="1-16" drill="0.4"/>
 <via x="13.9" y="13.6" extent="1-16" drill="0.4"/>
+<wire x1="24.35" y1="-1.75" x2="25.65" y2="-1.75" width="0.2286" layer="1"/>
+<wire x1="25.65" y1="-1.75" x2="25.7" y2="-1.8" width="0.2286" layer="1"/>
+<wire x1="25.7" y1="-1.8" x2="25.7" y2="-2.2" width="0.2286" layer="1"/>
+<wire x1="25.7" y1="-2.2" x2="25.8" y2="-2.3" width="0.2286" layer="1"/>
+<wire x1="13.1644" y1="3.2062" x2="13.1644" y2="3.3644" width="0.2286" layer="1"/>
 </signal>
 <signal name="+5V" class="1">
@@
 <wire x1="3.4" y1="-18.8" x2="8" y2="-18.8" width="0.254" layer="1"/>
 <wire x1="75.4" y1="7.6" x2="66.3" y2="7.6" width="0.3048" layer="1"/>
-<wire x1="66.3" y1="7.6" x2="60.8" y2="7.6" width="0.3048" layer="1"/>
-<wire x1="60.8" y1="7.6" x2="59.9" y2="6.7" width="0.3048" layer="1"/>
-<via x="59.9" y="6.7" extent="1-16" drill="0.4"/>
-<wire x1="59.9" y1="6.7" x2="30.7" y2="6.7" width="0.3048" layer="16"/>
+<wire x1="66.3" y1="7.6" x2="61.8" y2="7.6" width="0.3048" layer="1"/>
+<wire x1="61.8" y1="7.6" x2="60.9" y2="6.7" width="0.3048" layer="1"/>
+<via x="60.9" y="6.7" extent="1-16" drill="0.4"/>
+<wire x1="60.9" y1="6.7" x2="30.7" y2="6.7" width="0.3048" layer="16"/>
 <wire x1="30.7" y1="6.7" x2="30.5" y2="6.5" width="0.3048" layer="16"/>
 <wire x1="30.5" y1="6.5" x2="30.2" y2="6.2" width="0.3048" layer="16"/>
@@
 <contactref element="IC3" pad="50"/>
 <wire x1="19.6644" y1="15.2062" x2="19.6644" y2="14.2644" width="0.2286" layer="1"/>
-<wire x1="19.6644" y1="14.2644" x2="18.7" y2="13.3" width="0.2286" layer="1"/>
-<via x="18.7" y="13.3" extent="1-16" drill="0.4"/>
-<wire x1="18.7" y1="13.3" x2="20.2" y2="11.8" width="0.2286" layer="16"/>
-<wire x1="20.2" y1="11.8" x2="23.8" y2="11.8" width="0.2286" layer="16"/>
-<wire x1="23.8" y1="11.8" x2="26.9" y2="8.7" width="0.2286" layer="16"/>
+<wire x1="19.6644" y1="14.2644" x2="19" y2="13.5" width="0.2286" layer="1"/>
+<via x="19" y="13.5" extent="1-16" drill="0.4"/>
+<wire x1="19" y1="13.5" x2="20.5" y2="12" width="0.2286" layer="16"/>
+<wire x1="20.5" y1="12" x2="23.6" y2="12" width="0.2286" layer="16"/>
+<wire x1="23.6" y1="12" x2="26.9" y2="8.7" width="0.2286" layer="16"/>
 <wire x1="26.9" y1="8.7" x2="52.8" y2="8.7" width="0.2286" layer="16"/>
 <wire x1="52.8" y1="8.7" x2="54.2" y2="8.7" width="0.2286" layer="16"/>
@@
 <via x="35.3" y="-20.8" extent="1-16" drill="0.4"/>
 <wire x1="35.3" y1="-20.8" x2="35.3" y2="-20.4" width="0.3048" layer="16"/>
-<wire x1="35.3" y1="-20.4" x2="32.9" y2="-18" width="0.3048" layer="16"/>
-<wire x1="32.9" y1="-18" x2="22.7" y2="-18" width="0.3048" layer="16"/>
-<wire x1="22.7" y1="-18" x2="19.5" y2="-14.8" width="0.3048" layer="16"/>
+<wire x1="35.3" y1="-20.4" x2="33.4" y2="-18.5" width="0.3048" layer="16"/>
+<wire x1="33.4" y1="-18.5" x2="21" y2="-18.5" width="0.3048" layer="16"/>
+<wire x1="21" y1="-18.5" x2="20.2" y2="-17.7" width="0.3048" layer="16"/>
+<wire x1="20.2" y1="-17.7" x2="20.2" y2="-15.5" width="0.3048" layer="16"/>
+<wire x1="20.2" y1="-15.5" x2="19.5" y2="-14.8" width="0.3048" layer="16"/>
 <wire x1="19.5" y1="-14.8" x2="18.3" y2="-14.8" width="0.3048" layer="16"/>
 <wire x1="18.3" y1="-14.8" x2="15.2" y2="-17.9" width="0.3048" layer="16"/>
@@
 <wire x1="23.25" y1="-6.75" x2="23.2" y2="-6.8" width="0.254" layer="1"/>
 <via x="23.2" y="-6.8" extent="1-16" drill="0.6"/>
-<wire x1="23.2" y1="-6.8" x2="23.2" y2="-15.4" width="0.3048" layer="16"/>
-<wire x1="23.2" y1="-15.4" x2="23.4" y2="-15.6" width="0.3048" layer="16"/>
-<via x="23.4" y="-15.6" extent="1-16" drill="0.6"/>
-<wire x1="23.4" y1="-15.6" x2="23.4" y2="-18.9" width="0.3048" layer="1"/>
-<wire x1="23.4" y1="-18.9" x2="22.7" y2="-19.6" width="0.3048" layer="1"/>
+<wire x1="23.2" y1="-6.8" x2="23.2" y2="-14.1" width="0.3048" layer="16"/>
+<wire x1="23.2" y1="-14.1" x2="24.5" y2="-15.3" width="0.3048" layer="16"/>
+<via x="24.5" y="-15.3" extent="1-16" drill="0.6"/>
+<wire x1="24.5" y1="-15.3" x2="24.5" y2="-17.8" width="0.3048" layer="1"/>
+<wire x1="24.5" y1="-17.8" x2="22.7" y2="-19.6" width="0.3048" layer="1"/>
 <wire x1="22.7" y1="-19.6" x2="21.5" y2="-19.6" width="0.3048" layer="1"/>
 <wire x1="20.5106" y1="-5.72" x2="21.82" y2="-5.72" width="0.254" layer="1"/>

Commit message: routing
Connections:
- removed net N$23: IC1.19
- new net CHG: IC1.19, IC3.16
- net EN2: now also IC3.14
- net LED0: now also IC3.9
- net LED2: now also IC3.11
Routing:
- net LED2: track 0.00 -> 60.6 mm, vias 0 -> 4
- net LED0: track 0.00 -> 44.1 mm, vias 0 -> 4
- net EN2: track 4.31 -> 47.5 mm, vias 0 -> 4
- net CHG: track 0.00 -> 37.2 mm, vias 0 -> 4
- net N$23: track 3.49 -> 0.00 mm
- net VLIPO: track 63.9 -> 67.3 mm
- net VOLTAGE: track 0.00 -> 2.77 mm
- net +3V3: track 211.0 -> 210.4 mm

Commit message: routing
Connections:
- net LED1: now also IC3.54
- net LED3: now also IC3.55
Routing:
- net LED3: track 0.00 -> 112.2 mm, vias 0 -> 4
- net LED1: track 0.15 -> 61.7 mm, vias 0 -> 2
- net SS3: track 14.9 -> 13.8 mm
- net LED2: track 60.6 -> 59.7 mm
- net SW3: track 27.1 -> 26.4 mm
- net GND: vias 119 -> 127

Commit message: routing
Connections:
- net SCL: now also IC3.58
- net SDA: now also IC3.59
- net SW3: now also IC3.56; no longer IC3.59
Routing:
- net SCL: track 5.56 -> 64.0 mm, vias 0 -> 2
- net SDA: track 6.09 -> 63.1 mm, vias 0 -> 2
- net GND: track 79.7 -> 78.5 mm, vias 127 -> 129
- net SW3: track 26.4 -> 27.2 mm
