File: eagle/lun1k_v1_3.brd (EAGLE design)
At the start: 127.6 x 60.4 mm, 108 parts, among them IC1 LTC3558, IC2 LM27313, IC3 STM32F405RGT, IC4 NRF24L01SMD, J2 XF2-3015-1LW, Q1 Q12M-SMD-S, Q2 3.2X2.5CRYSTAL, SW1 JS102011SAQN, SW2 SWITCH_MCTAEF, SW3 SWITCH_MCTAEF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

Commit message: flash_db & adc & pcb misc
Parts:
- added C27: calculate for good oversampling performance, SparkFun-Capacitors:0402-CAP
- moved SW4 1.21 mm to (-2.60, -14.4)
- moved SW3 0.67 mm to (-0.30, -20.4)
- moved C39 0.51 mm to (14.2, 0.84)
- moved SW2 0.36 mm to (2.20, -27.1)
Connections:
- net GND: now also C27.1
- net VOLTAGE: now also C27.2
Routing:
- net 3.3V: track 307.8 -> 300.3 mm
- net GND: track 84.9 -> 88.0 mm
- net VOLTAGE: track 2.37 -> 3.57 mm
- net SW4: track 32.2 -> 33.0 mm
- net SW3: track 56.7 -> 57.4 mm
- net INTN: track 21.1 -> 20.5 mm
Other:
- board text added: "lun1k v1.3"
- board text removed: "lun1k v1.2"

Commit message: v1.3 updates
Parts:
- added U$3: MAKE-DD_LOGO'PROMPT', seb:MAKE-DD_LOGO_PROMPT
- moved R19 0.20 mm to (21.2, -9.80)
- moved R7 0.10 mm to (11.5, 1.10)
Connections:
- removed net EN2: IC1.15, R24.2, SW1.3
- new net LIPO_SWITCHED: IC1.15, R24.2, R6.2, SW1.3
- net VLIPO: no longer R6.2
Routing:
- net LIPO_SWITCHED: track 0.00 -> 61.9 mm, vias 0 -> 8
- net EN2: track 25.1 -> 0.00 mm, vias 2 -> 0
- net CHG: track 43.8 -> 41.4 mm
- net VLIPO: track 110.1 -> 107.9 mm, vias 9 -> 7
- net GND: track 88.0 -> 89.5 mm, vias 170 -> 171
- net N$15: track 24.9 -> 25.4 mm
