File: eagle/lun1k_v1_3.sch (EAGLE design)
At the start: 108 parts, among them IC1 LTC3558, IC2 LM27313, IC3 STM32F405RGT, IC4 NRF24L01SMD, J2 XF2-3015-1LW, Q1 Q12M-SMD-S, Q2 3.2X2.5CRYSTAL, SW1 JS102011SAQN, SW2 SWITCH_MCTAEF, SW3 SWITCH_MCTAEF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

Commit message: flash_db & adc & pcb misc
Parts:
- added C27: calculate for good oversampling performance, SparkFun-Capacitors:CAP0402-CAP
Connections:
- net GND: now also C27.1
- net VOLTAGE: now also C27.2
Changed lines of the file:
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@@
 <?xml version="1.0" encoding="utf-8"?>
 <!DOCTYPE eagle SYSTEM "eagle.dtd">
-<eagle version="6.4">
+<eagle version="6.6.0">
 <drawing>
 <settings>
@@
 <part name="R32" library="SparkFun-Passives" deviceset="RESISTOR" device="0402-RES" value="15k"/>
 <part name="GND46" library="supply1" deviceset="GND" device=""/>
+<part name="C27" library="SparkFun-Capacitors" deviceset="CAP" device="0402-CAP" value="calculate for good oversampling performance"/>
+<part name="GND47" library="supply1" deviceset="GND" device=""/>
 </parts>
 <sheets>
@@
 </instance>
 <instance part="GND46" gate="1" x="162.56" y="167.64"/>
+<instance part="C27" gate="G$1" x="154.94" y="226.06" rot="R180"/>
+<instance part="GND47" gate="1" x="154.94" y="215.9"/>
 </instances>
 <busses>
@@
 <pinref part="GND46" gate="1" pin="GND"/>
 </segment>
+<segment>
+<pinref part="GND47" gate="1" pin="GND"/>
+<pinref part="C27" gate="G$1" pin="1"/>
+<wire x1="154.94" y1="218.44" x2="154.94" y2="220.98" width="0.1524" layer="91"/>
+</segment>
 </net>
 <net name="+5V" class="1">
@@
 <wire x1="139.7" y1="231.14" x2="139.7" y2="233.68" width="0.1524" layer="91"/>
 <wire x1="139.7" y1="233.68" x2="139.7" y2="236.22" width="0.1524" layer="91"/>
-<wire x1="139.7" y1="233.68" x2="157.48" y2="233.68" width="0.1524" layer="91"/>
+<wire x1="139.7" y1="233.68" x2="154.94" y2="233.68" width="0.1524" layer="91"/>
 <junction x="139.7" y="233.68"/>
 <label x="149.86" y="233.68" size="1.778" layer="95"/>
 <pinref part="R7" gate="G$1" pin="2"/>
 <pinref part="R6" gate="G$1" pin="1"/>
-</segment>
-<segment>
+<pinref part="C27" gate="G$1" pin="2"/>
+<wire x1="154.94" y1="233.68" x2="157.48" y2="233.68" width="0.1524" layer="91"/>
+<wire x1="154.94" y1="228.6" x2="154.94" y2="233.68" width="0.1524" layer="91"/>
+<junction x="154.94" y="233.68"/>
+</segment>
+<segment>

Commit message: v1.3 updates
Parts:
- added U$3: MAKE-DD_LOGO'PROMPT', seb:MAKE-DD_LOGO'PROMPT'
Connections:
- removed net EN2: IC1.EN2, R24.2, SW1.3
- new net LIPO_SWITCHED: IC1.EN2, R24.2, R6.2, SW1.3
- net VLIPO: no longer R6.2
Changed lines of the file:
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@@
 <part name="C27" library="SparkFun-Capacitors" deviceset="CAP" device="0402-CAP" value="calculate for good oversampling performance"/>
 <part name="GND47" library="supply1" deviceset="GND" device=""/>
+<part name="U$3" library="seb" deviceset="MAKE-DD_LOGO" device="'PROMPT'"/>
 </parts>
 <sheets>
@@
 <instance part="C27" gate="G$1" x="154.94" y="226.06" rot="R180"/>
 <instance part="GND47" gate="1" x="154.94" y="215.9"/>
+<instance part="U$3" gate="G$1" x="147.32" y="111.76"/>
 </instances>
 <busses>
@@
 </segment>
 <segment>
-<wire x1="139.7" y1="246.38" x2="139.7" y2="251.46" width="0.1524" layer="91"/>
-<pinref part="R6" gate="G$1" pin="2"/>
-<label x="139.7" y="248.92" size="1.778" layer="95"/>
-</segment>
-<segment>
 <pinref part="IC1" gate="G$1" pin="BAT"/>
 <wire x1="302.26" y1="248.92" x2="297.18" y2="248.92" width="0.1524" layer="91"/>
@@
 </segment>
 </net>
-<net name="EN2" class="0">
+<net name="LIPO_SWITCHED" class="0">
 <segment>
 <wire x1="251.46" y1="193.04" x2="246.38" y2="193.04" width="0.1524" layer="91"/>
@@
 <pinref part="R24" gate="G$1" pin="2"/>
 <pinref part="SW1" gate="SW1" pin="3"/>
-<wire x1="223.52" y1="193.04" x2="246.38" y2="193.04" width="0.1524" layer="91"/>
+<wire x1="223.52" y1="193.04" x2="226.06" y2="193.04" width="0.1524" layer="91"/>
 <junction x="246.38" y="193.04"/>
-</segment>
-</net>
+<wire x1="226.06" y1="193.04" x2="246.38" y2="193.04" width="0.1524" layer="91"/>
+<wire x1="226.06" y1="193.04" x2="226.06" y2="187.96" width="0.1524" layer="91"/>
+<junction x="226.06" y="193.04"/>
+<wire x1="226.06" y1="187.96" x2="208.28" y2="187.96" width="0.1524" layer="91"/>
+<label x="208.28" y="187.96" size="1.778" layer="95"/>
+</segment>
+<segment>
+<wire x1="139.7" y1="246.38" x2="139.7" y2="251.46" width="0.1524" layer="91"/>
+<pinref part="R6" gate="G$1" pin="2"/>
+<label x="139.7" y="248.92" size="1.778" layer="95"/>
+</segment>
+</net>
