File: eagle/lun1k_v1_2.sch (EAGLE design)
At the start: 107 parts, among them IC1 LTC3558, IC2 LM27313, IC3 STM32F405RGT, IC4 NRF24L01SMD, J2 XF2-3015-1LW, Q1 Q12M-SMD-S, Q2 3.2X2.5CRYSTAL, SW1 JS102011SAQN, SW2 SWITCH_MCTAEF, SW3 SWITCH_MCTAEF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

Commit message: cap
Parts:
- added C27: 22pF, SparkFun-Capacitors:CAP0402-CAP
Connections:
- net GND: now also C27.1
- net VOLTAGE: now also C27.2
Changed lines of the file:
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@@
 <?xml version="1.0" encoding="utf-8"?>
 <!DOCTYPE eagle SYSTEM "eagle.dtd">
-<eagle version="6.2">
+<eagle version="6.6.0">
 <drawing>
 <settings>
@@
 <part name="Q3" library="microbuilder" deviceset="MOSFET-P" device=""/>
 <part name="R26" library="rcl" deviceset="R-EU_" device="R0402" value="15k"/>
+<part name="C27" library="SparkFun-Capacitors" deviceset="CAP" device="0402-CAP" value="22pF"/>
+<part name="GND46" library="supply1" deviceset="GND" device=""/>
 </parts>
 <sheets>
@@
 <instance part="Q3" gate="G$1" x="162.56" y="-17.78"/>
 <instance part="R26" gate="G$1" x="152.4" y="-10.16" rot="R90"/>
+<instance part="C27" gate="G$1" x="152.4" y="228.6" smashed="yes" rot="R180">
+<attribute name="NAME" x="149.479" y="222.504" size="1.778" layer="95" rot="R90"/>
+<attribute name="VALUE" x="157.099" y="222.504" size="1.778" layer="96" rot="R90"/>
+</instance>
+<instance part="GND46" gate="1" x="152.4" y="215.9"/>
 </instances>
 <busses>
@@
 <pinref part="GND44" gate="1" pin="GND"/>
 </segment>
+<segment>
+<pinref part="C27" gate="G$1" pin="1"/>
+<wire x1="152.4" y1="223.52" x2="152.4" y2="218.44" width="0.1524" layer="91"/>
+<pinref part="GND46" gate="1" pin="GND"/>
+</segment>
 </net>
 <net name="+5V" class="1">
@@
 <wire x1="139.7" y1="231.14" x2="139.7" y2="233.68" width="0.1524" layer="91"/>
 <wire x1="139.7" y1="233.68" x2="139.7" y2="236.22" width="0.1524" layer="91"/>
-<wire x1="139.7" y1="233.68" x2="157.48" y2="233.68" width="0.1524" layer="91"/>
+<wire x1="139.7" y1="233.68" x2="152.4" y2="233.68" width="0.1524" layer="91"/>
 <junction x="139.7" y="233.68"/>
 <label x="149.86" y="233.68" size="1.778" layer="95"/>
 <pinref part="R7" gate="G$1" pin="2"/>
 <pinref part="R6" gate="G$1" pin="1"/>
-</segment>
-<segment>
+<pinref part="C27" gate="G$1" pin="2"/>
+<wire x1="152.4" y1="233.68" x2="157.48" y2="233.68" width="0.1524" layer="91"/>
+<wire x1="152.4" y1="231.14" x2="152.4" y2="233.68" width="0.1524" layer="91"/>
+<junction x="152.4" y="233.68"/>
+</segment>
+<segment>
